File: PCB Files/LTE Shield v2.brd (EAGLE design)
At the start: 58.4 x 53.3 mm, 47 parts, among them IC1 TXB0104, IC2 MCP9808, IC3 MCP73831, J5 microUSB, J6 LiPo, Q1 FDV301N, Q2 FDV301N, X1 LTE-uFL, X2 GNSS-uFL

Commit message: Add files via upload
Parts:
- C1, C2: value 0.1uF -> 4.7uF
- C4: value 4.7uF -> 0.1uF
- C5: value 0.22uF -> 0.1uF
- C6: value 33pF -> 0.22uF
- C7: value 4.7uF -> 33pF
- IC1: value TXB0104 -> MCP73831; device TimWoo-IC:VQFN-14 -> TimWoo-IC:SOT23-5
- IC2: value MCP9808 -> TXB0104; device TimWoo-IC:8-TSSOP -> TimWoo-IC:VQFN-14
- IC3: value MCP73831 -> MCP9808; device TimWoo-IC:SOT23-5 -> TimWoo-IC:8-TSSOP
- J5: value microUSB -> LiPo; device TimWoo-Connectors:USB-B-MICRO-SMD -> TimWoo-Connectors:JST-2-SMD
- J6: value LiPo -> microUSB; device TimWoo-Connectors:JST-2-SMD -> TimWoo-Connectors:USB-B-MICRO-SMD
- R1, R2: value 10k -> 1k
- R3: value 10k -> 2k
- R4: device TimWoo-Resistors:RES_ARRAY_4X0603 -> TimWoo-Resistors:0603-RES-MARKED
- R5, R6: value 1k -> 10k
- R7: value 2k -> 10k; device TimWoo-Resistors:0603-RES-MARKED -> TimWoo-Resistors:RES_ARRAY_4X0603
- moved FID1 54.8 mm to (45.7, 44.5)
- moved FID2 54.8 mm to (5.08, 7.62)
- moved R5 42.0 mm to (13.0, 43.7), turned to 0 degrees
- moved JP1 41.8 mm to (17.8, 5.33)
- moved JP2 41.8 mm to (21.3, 47.0)
- moved R3 39.5 mm to (31.2, 6.99)
- moved R2 38.5 mm to (32.1, 10.3), turned to 270 degrees
- moved R1 37.1 mm to (34.8, 7.75), turned to 180 degrees
- moved R6 37.0 mm to (13.1, 42.0), turned to 0 degrees
- moved C4 36.4 mm to (31.1, 44.3), turned to 180 degrees
- moved IC3 36.0 mm to (9.65, 39.9)
- moved C2 35.6 mm to (24.9, 9.27), turned to 270 degrees
- moved R7 35.2 mm to (9.65, 34.8)
- moved C1 34.4 mm to (26.9, 8.13), turned to 90 degrees
- moved IC1 34.1 mm to (29.5, 9.78), turned to 180 degrees
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Connections:
- net 1.8V: now also C3.2, IC2.1, IC2.8; no longer C1.2, IC1.1, IC1.8
- net 5V: now also C1.1, C5.1, IC1.4, IC2.14, IC3.8, R4.2, R6.2; no longer C2.1, C3.1, IC1.14, IC2.8, IC3.4, R2.2, R3.2
- net ADDR0: now also IC3.7, R7.6; no longer IC2.7, R4.6
- net ADDR1: now also IC3.6, R7.7; no longer IC2.6, R4.7
- net ADDR2: now also IC3.5, R7.8; no longer IC2.5, R4.8
- net ALERT: now also IC3.3, JP2.2, R4.1; no longer IC2.3, JP1.2, R1.1
- net D+: now also J6.D+; no longer J5.D+
- net D-: now also J6.D-; no longer J5.D-
- net GND: now also C1.2, C3.1, C6.2, IC1.2, IC2.11, IC2.7, IC2.PAD, IC3.4, J5.1, J6.GND, J6.SHIELD1, J6.SHIELD2, J6.SHIELD3, R3.2, R7.1, R7.3; no longer C1.1, C3.2, C7.2, IC1.11, IC1.4, IC1.7, IC1.PAD, IC3.2, J5.GND, J5.SHIELD1, J5.SHIELD2, J5.SHIELD3, J6.1, R4.1, R4.2, R4.3
- net LTE_RI: now also IC2.5; no longer IC1.5
- net LTE_RXD: now also IC2.2; no longer IC1.2
- net LTE_TXD: now also IC2.3; no longer IC1.3
- net N$1: now also C7.2; no longer C6.2
- net N$3: now also C7.1; no longer C6.1
- net N$6: now also R1.1; no longer R5.1
- net N$7: now also JP2.1; no longer JP1.1
- net N$8: now also R2.2; no longer R6.2
- net N$9: now also JP1.2; no longer JP2.2
- net PROG: now also IC1.5, R3.1; no longer IC3.5, R7.1
- net SCL: now also IC3.2, R5.1; no longer IC2.2, R2.1
- net SDA: now also IC3.1, R6.1; no longer IC2.1, R3.1
- net SIM_VCC: now also C6.1; no longer C5.1
- net STAT: now also IC1.1, R2.1; no longer IC3.1, R6.1
- net UC_RI: now also IC2.10; no longer IC1.10
- net UC_RXD: now also IC2.13; no longer IC1.13
- net UC_TXD: now also IC2.12; no longer IC1.12
- net VBAT: now also C2.1, IC1.3, J5.2, JP1.1; no longer C7.1, IC3.3, J6.2, JP2.1
- net V_USB: now also J6.VBUS; no longer J5.VBUS

Commit message: Add files via upload
Routing:
- net N$10: track 0.00 -> 2.52 mm
- net N$11: track 0.00 -> 2.41 mm
- net GND: vias 75 -> 74
Changed lines of the file:
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@@
 <?xml version="1.0" encoding="utf-8"?>
 <!DOCTYPE eagle SYSTEM "eagle.dtd">
-<eagle version="8.4.1">
+<eagle version="8.4.2">
 <drawing>
 <settings>
@@
 <layer number="23" name="tOrigins" color="15" fill="1" visible="yes" active="yes"/>
 <layer number="24" name="bOrigins" color="15" fill="1" visible="yes" active="yes"/>
-<layer number="25" name="tNames" color="7" fill="1" visible="no" active="yes"/>
-<layer number="26" name="bNames" color="7" fill="1" visible="no" active="yes"/>
+<layer number="25" name="tNames" color="7" fill="1" visible="yes" active="yes"/>
+<layer number="26" name="bNames" color="7" fill="1" visible="yes" active="yes"/>
 <layer number="27" name="tValues" color="7" fill="1" visible="no" active="yes"/>
 <layer number="28" name="bValues" color="7" fill="1" visible="no" active="yes"/>
@@
 <text x="0" y="57.15" size="2.54" layer="51" font="vector" ratio="16">Designed by Timothy Woo
 Released under CC-BY-SA-4.0 license</text>
-<text x="16.383" y="4.064" size="0.8128" layer="22" font="vector" ratio="16" rot="R90">VBAT</text>
 <text x="18.415" y="4.318" size="1.27" layer="21" font="vector" ratio="16" rot="R90">VBAT*</text>
+<text x="19.177" y="6.858" size="0.8128" layer="22" font="vector" ratio="16" rot="MR0">VBAT</text>
 </plain>
 <attributes>
@@
 </element>
 <element name="C6" library="TimWoo-Capacitors" package="0603-CAP-MARKED" value="0.22uF" x="17.78" y="14.986" smashed="yes">
-<attribute name="NAME" x="17.526" y="16.002" size="0.4064" layer="25" font="vector" ratio="16"/>
+<attribute name="NAME" x="18.288" y="13.97" size="0.8128" layer="25" font="vector" ratio="16" rot="R180"/>
 <attribute name="VALUE" x="16.764" y="13.843" size="0.4064" layer="27" font="vector"/>
 </element>
 <element name="D3" library="TimWoo-Diodes" library_urn="urn:adsk.eagle:library:501758" package="SOT-353" value="MSQA6V1W5T2G" x="17.145" y="19.177" smashed="yes" rot="R180">
-<attribute name="NAME" x="17.399" y="18.288" size="0.4064" layer="25" font="vector" ratio="16" rot="R180"/>
+<attribute name="NAME" x="17.907" y="17.526" size="0.8128" layer="25" font="vector" ratio="16" rot="R180"/>
 <attribute name="VALUE" x="18.161" y="20.955" size="0.4064" layer="27" font="vector" ratio="16" rot="R180"/>
 </element>
@@
 </element>
 <element name="R9" library="TimWoo-Resistors" library_urn="urn:adsk.eagle:library:500711" package="0603-RES-MARKED" package3d_urn="urn:adsk.eagle:package:500751/2" value="470" x="47.117" y="11.938" smashed="yes" rot="R180">
-<attribute name="NAME" x="49.022" y="11.684" size="0.8128" layer="25" font="vector" ratio="16"/>
+<attribute name="NAME" x="45.212" y="12.319" size="0.8128" layer="25" font="vector" ratio="16" rot="R180"/>
 <attribute name="VALUE" x="48.133" y="13.208" size="0.4064" layer="27" font="vector" ratio="16" rot="R180"/>
 </element>
@@
 </element>
 <element name="LED1" library="TimWoo-LED" library_urn="urn:adsk.eagle:library:501982" package="LED-0603-MARKED" package3d_urn="urn:adsk.eagle:package:502010/2" value="Green" x="34.798" y="9.398" smashed="yes">
-<attribute name="NAME" x="40.64" y="9.017" size="0.8128" layer="25" font="vector" ratio="16"/>
+<attribute name="NAME" x="38.608" y="8.001" size="0.8128" layer="25" font="vector" ratio="16"/>
 <attribute name="VALUE" x="33.782" y="8.001" size="0.4064" layer="27"/>
 </element>
@@
 <contactref element="R7" pad="2"/>
 <contactref element="R7" pad="3"/>
-<via x="9.652" y="39.878" extent="1-16" drill="0.508" diameter="1.016"/>
 <via x="7.112" y="42.418" extent="1-16" drill="0.508" diameter="1.016"/>
 <via x="7.112" y="39.878" extent="1-16" drill="0.508" diameter="1.016"/>
@@
 <contactref element="Q2" pad="3"/>
 <contactref element="R9" pad="1"/>
-<wire x1="47.967" y1="11.938" x2="48.217" y2="14.351" width="0" layer="19" extent="1-1"/>
+<wire x1="48.217" y1="14.351" x2="48.217" y2="13.165" width="0.3048" layer="1"/>
+<wire x1="48.006" y1="12.954" x2="48.006" y2="11.977" width="0.3048" layer="1"/>
+<wire x1="48.006" y1="11.977" x2="47.967" y2="11.938" width="0.3048" layer="1"/>
+<wire x1="48.217" y1="13.165" x2="48.006" y2="12.954" width="0.3048" layer="1"/>
 </signal>
 <signal name="N$11">
 <contactref element="R9" pad="2"/>
 <contactref element="LED4" pad="C"/>
-<wire x1="47.994" y1="10.287" x2="46.267" y2="11.938" width="0" layer="19" extent="1-1"/>
+<wire x1="46.267" y1="11.938" x2="46.343" y2="11.938" width="0.3048" layer="1"/>
+<wire x1="46.343" y1="11.938" x2="47.994" y2="10.287" width="0.3048" layer="1"/>
 </signal>
 </signals>

Commit message: Add files via upload
Parts:
- added JP3: (no value), TimWoo-Connectors:SMT-JUMPER_2_NC_TRACE_SILK
- moved FID1 2.54 mm to (48.3, 44.5)
Connections:
- new net LTE_DTR: IC2.5, U1.3
- new net N$12: JP3.2, LED3.A
- new net UC_DTR: IC2.10, J4.5
- net GND: no longer IC2.11, IC2.4
- net LTE_PWR: now also J4.4; no longer J4.5
- net LTE_RI: now also IC2.4; no longer IC2.5
- net UC_RI: now also IC2.11; no longer IC2.10
- net VBAT: now also JP3.1; no longer LED3.A
Routing:
- net UC_DTR: track 0.00 -> 10.3 mm
- net LTE_DTR: track 0.00 -> 5.83 mm
- net VBAT: track 96.1 -> 98.9 mm
- net N$12: track 0.00 -> 2.42 mm
- net LTE_PWR: track 8.63 -> 9.69 mm
- net UC_RI: track 7.72 -> 8.67 mm
Changed lines of the file:
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@@
 </element>
 <element name="FID2" library="TimWoo-Aesthetics" library_urn="urn:adsk.eagle:library:502097" package="FIDUCIAL_1MM" package3d_urn="urn:adsk.eagle:package:502130/2" value="FIDUCIAL" x="5.08" y="7.62" smashed="yes"/>
-<element name="FID1" library="TimWoo-Aesthetics" library_urn="urn:adsk.eagle:library:502097" package="FIDUCIAL_1MM" package3d_urn="urn:adsk.eagle:package:502130/2" value="FIDUCIAL" x="45.72" y="44.45" smashed="yes"/>
+<element name="FID1" library="TimWoo-Aesthetics" library_urn="urn:adsk.eagle:library:502097" package="FIDUCIAL_1MM" package3d_urn="urn:adsk.eagle:package:502130/2" value="FIDUCIAL" x="48.26" y="44.45" smashed="yes"/>
 <element name="IC1" library="TimWoo-IC" package="SOT23-5" value="MCP73831" x="29.464" y="9.779" smashed="yes" rot="R180">
 <attribute name="NAME" x="28.575" y="9.398" size="0.8128" layer="25" font="vector" ratio="16"/>
@@
 <element name="Q1" library="TimWoo-MOSFETs" library_urn="urn:adsk.eagle:library:501962" package="SOT23-3" package3d_urn="urn:adsk.eagle:package:501973/2" value="FDV301N" x="47.244" y="36.322" rot="R90"/>
 <element name="Q2" library="TimWoo-MOSFETs" library_urn="urn:adsk.eagle:library:501962" package="SOT23-3" package3d_urn="urn:adsk.eagle:package:501973/2" value="FDV301N" x="47.117" y="14.351" rot="R270"/>
+<element name="JP3" library="TimWoo-Connectors" library_urn="urn:adsk.eagle:library:500889" package="SMT-JUMPER_2_NC_TRACE_SILK" package3d_urn="urn:adsk.eagle:package:501668/1" value="" x="45.72" y="42.799" smashed="yes" rot="R180">
+<attribute name="NAME" x="45.72" y="44.069" size="0.6096" layer="25" font="vector" ratio="20" align="bottom-center"/>
+<attribute name="VALUE" x="45.72" y="43.942" size="0.6096" layer="27" font="vector" ratio="20" rot="R180" align="top-center"/>
+</element>
 </elements>
 <signals>
@@
 <contactref element="J3" pad="7"/>
 <contactref element="LED1" pad="C"/>
-<contactref element="IC2" pad="4"/>
-<contactref element="IC2" pad="11"/>
 <wire x1="4.757" y1="29.18" x2="5.999" y2="29.18" width="0.4064" layer="1"/>
 <via x="2.032" y="30.48" extent="1-16" drill="0.508" diameter="1.016"/>
@@
 <wire x1="45.02" y1="20.955" x2="45.02" y2="20.4" width="0.508" layer="1"/>
 <wire x1="45.02" y1="21.4" x2="45.02" y2="21.844" width="2.032" layer="1"/>
-<wire x1="42.799" y1="21.336" x2="44.639" y2="21.336" width="1.905" layer="1"/>
+<wire x1="44.639" y1="21.336" x2="42.799" y2="21.336" width="1.905" layer="1"/>
 <wire x1="44.639" y1="21.336" x2="45.02" y2="20.955" width="2.032" layer="1"/>
 <wire x1="45.02" y1="21.4" x2="45.02" y2="20.955" width="1.905" layer="1"/>
@@
 <wire x1="17.78" y1="5.7404" x2="17.78" y2="6.096" width="0.6096" layer="16"/>
 <wire x1="17.78" y1="6.096" x2="17.78" y2="7.62" width="1.016" layer="16"/>
-<contactref element="LED3" pad="A"/>
 <contactref element="LED4" pad="A"/>
 <wire x1="46.24" y1="10.287" x2="45.593" y2="10.287" width="0.3048" layer="1"/>
 <wire x1="42.799" y1="13.081" x2="42.799" y2="21.336" width="0.3048" layer="1"/>
 <wire x1="45.593" y1="10.287" x2="42.799" y2="13.081" width="0.3048" layer="1"/>
-<wire x1="46.24" y1="40.386" x2="45.466" y2="40.386" width="0.3048" layer="1"/>
-<wire x1="42.799" y1="37.719" x2="42.799" y2="21.336" width="0.3048" layer="1"/>
-<wire x1="45.466" y1="40.386" x2="42.799" y2="37.719" width="0.3048" layer="1"/>
+<contactref element="JP3" pad="1"/>
+<wire x1="42.799" y1="40.894" x2="44.704" y2="42.799" width="0.3048" layer="1"/>
+<wire x1="44.704" y1="42.799" x2="46.228" y2="42.799" width="0.3048" layer="1"/>
+<wire x1="42.799" y1="21.336" x2="42.799" y2="40.894" width="0.3048" layer="1"/>
 </signal>
 <signal name="STAT">
@@
 <signal name="LTE_RI">
 <contactref element="U1" pad="4"/>
-<contactref element="IC2" pad="5"/>
-<wire x1="35.933" y1="41.582" x2="35.933" y2="41.029" width="0.3048" layer="1"/>
-<wire x1="38.02" y1="38.942" x2="38.02" y2="37.4" width="0.3048" layer="1"/>
-<wire x1="35.933" y1="41.029" x2="38.02" y2="38.942" width="0.3048" layer="1"/>
+<contactref element="IC2" pad="4"/>
+<wire x1="38.02" y1="37.4" x2="38.02" y2="38.688" width="0.3048" layer="1"/>
+<wire x1="38.02" y1="38.688" x2="36.83" y2="39.751" width="0.3048" layer="1"/>
+<wire x1="36.83" y1="39.751" x2="36.449" y2="39.751" width="0.3048" layer="1"/>
+<wire x1="35.433" y1="40.767" x2="35.433" y2="41.582" width="0.3048" layer="1"/>
+<wire x1="36.449" y1="39.751" x2="35.433" y2="40.767" width="0.3048" layer="1"/>
 </signal>
 <signal name="LTE_RXD">
@@
 <signal name="LTE_PWR">
 <contactref element="D1" pad="C"/>
-<contactref element="J4" pad="5"/>
-<wire x1="43.18" y1="50.8" x2="41.021" y2="48.641" width="0.3048" layer="1"/>
-<wire x1="41.021" y1="48.641" x2="41.021" y2="43.06" width="0.3048" layer="1"/>
+<contactref element="J4" pad="4"/>
+<wire x1="41.021" y1="43.06" x2="41.021" y2="46.101" width="0.3048" layer="1"/>
+<wire x1="41.021" y1="46.101" x2="45.72" y2="50.8" width="0.3048" layer="1"/>
 </signal>
 <signal name="NETLIGHT">
@@
 <signal name="UC_RI">
 <contactref element="J4" pad="6"/>
-<contactref element="IC2" pad="10"/>
-<wire x1="35.933" y1="45.032" x2="35.933" y2="46.093" width="0.3048" layer="1"/>
-<wire x1="35.933" y1="46.093" x2="40.64" y2="50.8" width="0.3048" layer="1"/>
+<contactref element="IC2" pad="11"/>
+<wire x1="35.433" y1="45.032" x2="35.433" y2="46.863" width="0.3048" layer="1"/>
+<wire x1="35.433" y1="46.863" x2="37.465" y2="48.895" width="0.3048" layer="1"/>
+<wire x1="37.465" y1="48.895" x2="38.735" y2="48.895" width="0.3048" layer="1"/>
+<wire x1="38.735" y1="48.895" x2="40.64" y2="50.8" width="0.3048" layer="1"/>
 </signal>
 <signal name="5V">
@@
 <wire x1="46.343" y1="11.938" x2="47.994" y2="10.287" width="0.3048" layer="1"/>
 </signal>
+<signal name="LTE_DTR">
+<contactref element="U1" pad="3"/>
+<contactref element="IC2" pad="5"/>
+<wire x1="39.02" y1="37.4" x2="39.02" y2="38.577" width="0.3048" layer="1"/>
+<wire x1="37.338" y1="40.259" x2="36.703" y2="40.259" width="0.3048" layer="1"/>
+<wire x1="36.703" y1="40.259" x2="35.933" y2="41.029" width="0.3048" layer="1"/>
+<wire x1="35.933" y1="41.029" x2="35.933" y2="41.582" width="0.3048" layer="1"/>
+<wire x1="39.02" y1="38.577" x2="37.338" y2="40.259" width="0.3048" layer="1"/>
+</signal>
+<signal name="UC_DTR">
+<contactref element="IC2" pad="10"/>
+<contactref element="J4" pad="5"/>
+<wire x1="35.933" y1="45.032" x2="35.933" y2="46.22" width="0.3048" layer="1"/>
+<wire x1="35.933" y1="46.22" x2="37.973" y2="48.26" width="0.3048" layer="1"/>
+<wire x1="37.973" y1="48.26" x2="40.64" y2="48.26" width="0.3048" layer="1"/>
+<wire x1="40.64" y1="48.26" x2="43.18" y2="50.8" width="0.3048" layer="1"/>
+</signal>
+<signal name="N$12">
+<contactref element="JP3" pad="2"/>
+<contactref element="LED3" pad="A"/>
+<wire x1="46.24" y1="40.386" x2="46.24" y2="42.787" width="0.3048" layer="1"/>
+<wire x1="46.24" y1="42.787" x2="46.228" y2="42.799" width="0.3048" layer="1"/>
+</signal>
 </signals>
