File: PCB Files/LTE Shield v2.sch (EAGLE design)
At the start: 47 parts, among them IC1 TXB0104, IC2 MCP9808, IC3 MCP73831, J5 microUSB, J6 LiPo, Q1 FDV301N, Q2 FDV301N, X1 LTE-uFL, X2 GNSS-uFL

Commit message: Add files via upload
Parts:
- C1, C2: value 0.1uF -> 4.7uF
- C4: value 4.7uF -> 0.1uF
- C5: value 0.22uF -> 0.1uF
- C6: value 33pF -> 0.22uF
- C7: value 4.7uF -> 33pF
- IC1: value TXB0104 -> MCP73831; device TimWoo-IC:LEVEL_SHIFTER_TXB0104TXB0104RGYR -> TimWoo-IC:MCP73831
- IC2: value MCP9808 -> TXB0104; device TimWoo-IC:MCP9808-MSOP -> TimWoo-IC:LEVEL_SHIFTER_TXB0104TXB0104RGYR
- IC3: value MCP73831 -> MCP9808; device TimWoo-IC:MCP73831 -> TimWoo-IC:MCP9808-MSOP
- J5: value microUSB -> LiPo; device TimWoo-Connectors:MICRO-USB_SMD_NOSHIELDV1 -> TimWoo-Connectors:M02-JST-2MM-SMT
- J6: value LiPo -> microUSB; device TimWoo-Connectors:M02-JST-2MM-SMT -> TimWoo-Connectors:MICRO-USB_SMD_NOSHIELDV1
- R1, R2: value 10k -> 1k
- R3: value 10k -> 2k
- R4: device TimWoo-Resistors:RESISTOR_ARRAY_4X0603-ARV -> TimWoo-Resistors:RESISTORMARKED-0603
- R5, R6: value 1k -> 10k
- R7: value 2k -> 10k; device TimWoo-Resistors:RESISTORMARKED-0603 -> TimWoo-Resistors:RESISTOR_ARRAY_4X0603-ARV
Connections:
- net 1.8V: now also C3.2, IC2.OE, IC2.VCCA; no longer C1.2, IC1.OE, IC1.VCCA
- net 5V: now also C1.1, C5.1, IC1.VIN, IC2.VCCB, IC3.VDD, R4.2, R6.2; no longer C2.1, C3.1, IC1.VCCB, IC2.VDD, IC3.VIN, R2.2, R3.2
- net ADDR0: now also IC3.A0, R7C.2; no longer IC2.A0, R4C.2
- net ADDR1: now also IC3.A1, R7B.2; no longer IC2.A1, R4B.2
- net ADDR2: now also IC3.A2, R7A.2; no longer IC2.A2, R4A.2
- net ALERT: now also IC3.ALERT, JP2.2, R4.1; no longer IC2.ALERT, JP1.2, R1.1
- net D+: now also J6.D+; no longer J5.D+
- net D-: now also J6.D-; no longer J5.D-
- net GND: now also C1.2, C3.1, C6.2, IC1.VSS, IC2.A3, IC2.B3, IC3.GND, J5.2, J6.GND, R3.2, R7A.1, R7B.1, R7C.1; no longer C1.1, C3.2, C7.2, IC1.A3, IC1.B3, IC1.GND, IC3.VSS, J5.GND, J6.2, R4A.1, R4B.1, R4C.1, R7.2
- net LTE_RI: now also IC2.A4; no longer IC1.A4
- net LTE_RXD: now also IC2.A1; no longer IC1.A1
- net LTE_TXD: now also IC2.A2; no longer IC1.A2
- net N$1: now also C7.2; no longer C6.2
- net N$3: now also C7.1; no longer C6.1
- net N$6: now also R1.1; no longer R5.1
- net N$7: now also JP2.1; no longer JP1.1
- net N$8: now also R2.2; no longer R6.2
- net N$9: now also JP1.2; no longer JP2.2
- net PROG: now also IC1.PROG, R3.1; no longer IC3.PROG, R7.1
- net SCL: now also IC3.SCL, R5.1; no longer IC2.SCL, R2.1
- net SDA: now also IC3.SDA, R6.1; no longer IC2.SDA, R3.1
- net SIM_VCC: now also C6.1; no longer C5.1
- net STAT: now also IC1.STAT, R2.1; no longer IC3.STAT, R6.1
- net UC_RI: now also IC2.B4; no longer IC1.B4
- net UC_RXD: now also IC2.B1; no longer IC1.B1
- net UC_TXD: now also IC2.B2; no longer IC1.B2
- net VBAT: now also C2.1, IC1.VBAT, J5.1, JP1.1; no longer C7.1, IC3.VBAT, J6.1, JP2.1
- net V_USB: now also J6.VBUS; no longer J5.VBUS
Other:
- moved on the sheet: C1, C2, C3, C4, C5, C6, C7, JP1, JP2, R1, R2, R3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

Commit message: Add files via upload
Parts:
- added JP3: (no value), TimWoo-Connectors:JUMPER-SMT_2_NC_TRACE_SILK
Connections:
- new net LTE_DTR: IC2.A4, U1.DTR
- new net N$12: JP3.2, LED3.A
- new net UC_DTR: IC2.B4, J4.5
- net GND: no longer IC2.A3, IC2.B3
- net LTE_PWR: now also J4.4; no longer J4.5
- net LTE_RI: now also IC2.A3; no longer IC2.A4
- net UC_RI: now also IC2.B3; no longer IC2.B4
- net VBAT: now also JP3.1; no longer LED3.A
Other:
- note added: "Cut jumper to disable PWR LED"
Changed lines of the file:
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@@
 <?xml version="1.0" encoding="utf-8"?>
 <!DOCTYPE eagle SYSTEM "eagle.dtd">
-<eagle version="8.4.1">
+<eagle version="8.4.2">
 <drawing>
 <settings>
@@
 <part name="C11" library="TimWoo-Capacitors" library_urn="urn:adsk.eagle:library:500759" deviceset="CAP" device="1206" package3d_urn="urn:adsk.eagle:package:500778/1" value="150uF"/>
 <part name="GND29" library="TimWoo-Aesthetics" deviceset="GND" device=""/>
-<part name="GND12" library="TimWoo-Aesthetics" deviceset="GND" device=""/>
 <part name="C3" library="TimWoo-Capacitors" library_urn="urn:adsk.eagle:library:500759" deviceset="CAP" device="MARKED-0603" package3d_urn="urn:adsk.eagle:package:500792/2" value="0.1uF"/>
 <part name="C4" library="TimWoo-Capacitors" deviceset="CAP" device="MARKED-0603" value="0.1uF"/>
@@
 <part name="SUPPLY12" library="TimWoo-Aesthetics" deviceset="VBAT" device=""/>
 <part name="SUPPLY15" library="TimWoo-Aesthetics" deviceset="VBAT" device=""/>
+<part name="JP3" library="TimWoo-Connectors" library_urn="urn:adsk.eagle:library:500889" deviceset="JUMPER-SMT_2_NC_TRACE" device="_SILK" package3d_urn="urn:adsk.eagle:package:501668/1"/>
 </parts>
 <sheets>
@@
 <wire x1="233.68" y1="91.44" x2="431.8" y2="91.44" width="0.1524" layer="94" style="longdash"/>
 <text x="241.3" y="76.2" size="5.08" layer="94">SIM7000 Status LED's</text>
+<text x="254" y="58.42" size="1.778" layer="97">Cut jumper to
+disable PWR LED</text>
 </plain>
 <instances>
@@
 <instance part="C11" gate="G$1" x="408.94" y="223.52"/>
 <instance part="GND29" gate="1" x="393.7" y="213.36"/>
-<instance part="GND12" gate="1" x="203.2" y="218.44"/>
 <instance part="C3" gate="G$1" x="167.64" y="243.84" rot="R90"/>
 <instance part="C4" gate="G$1" x="210.82" y="243.84" rot="R90"/>
@@
 <instance part="Q1" gate="G$1" x="254" y="25.4"/>
 <instance part="Q2" gate="G$1" x="294.64" y="25.4"/>
-<instance part="SUPPLY12" gate="G$1" x="256.54" y="55.88"/>
+<instance part="SUPPLY12" gate="G$1" x="241.3" y="60.96"/>
 <instance part="SUPPLY15" gate="G$1" x="297.18" y="55.88"/>
+<instance part="JP3" gate="G$1" x="248.92" y="55.88"/>
 </instances>
 <busses>
@@
 <wire x1="175.26" y1="223.52" x2="172.72" y2="223.52" width="0.1524" layer="91"/>
 <wire x1="172.72" y1="223.52" x2="172.72" y2="220.98" width="0.1524" layer="91"/>
-<pinref part="IC2" gate="G$1" pin="A3"/>
-<wire x1="175.26" y1="231.14" x2="172.72" y2="231.14" width="0.1524" layer="91"/>
-<wire x1="172.72" y1="231.14" x2="172.72" y2="223.52" width="0.1524" layer="91"/>
-<junction x="172.72" y="223.52"/>
 </segment>
 <segment>
@@
 <wire x1="73.66" y1="30.48" x2="71.12" y2="30.48" width="0.1524" layer="91"/>
 <wire x1="71.12" y1="30.48" x2="71.12" y2="27.94" width="0.1524" layer="91"/>
-</segment>
-<segment>
-<pinref part="IC2" gate="G$1" pin="B3"/>
-<pinref part="GND12" gate="1" pin="GND"/>
-<wire x1="200.66" y1="231.14" x2="203.2" y2="231.14" width="0.1524" layer="91"/>
-<wire x1="203.2" y1="231.14" x2="203.2" y2="220.98" width="0.1524" layer="91"/>
 </segment>
 <segment>
@@
 </segment>
 <segment>
-<pinref part="LED3" gate="G$1" pin="A"/>
-<pinref part="SUPPLY12" gate="G$1" pin="VBAT"/>
-<wire x1="256.54" y1="55.88" x2="256.54" y2="53.34" width="0.1524" layer="91"/>
-</segment>
-<segment>
 <pinref part="LED4" gate="G$1" pin="A"/>
 <pinref part="SUPPLY15" gate="G$1" pin="VBAT"/>
 <wire x1="297.18" y1="55.88" x2="297.18" y2="53.34" width="0.1524" layer="91"/>
+</segment>
+<segment>
+<pinref part="JP3" gate="G$1" pin="1"/>
+<wire x1="243.84" y1="55.88" x2="241.3" y2="55.88" width="0.1524" layer="91"/>
+<pinref part="SUPPLY12" gate="G$1" pin="VBAT"/>
+<wire x1="241.3" y1="55.88" x2="241.3" y2="60.96" width="0.1524" layer="91"/>
 </segment>
 </net>
@@
 </segment>
 <segment>
-<pinref part="IC2" gate="G$1" pin="A4"/>
-<wire x1="175.26" y1="228.6" x2="170.18" y2="228.6" width="0.1524" layer="91"/>
-<label x="170.18" y="228.6" size="1.27" layer="95" rot="R180" xref="yes"/>
+<pinref part="IC2" gate="G$1" pin="A3"/>
+<wire x1="175.26" y1="231.14" x2="172.72" y2="231.14" width="0.1524" layer="91"/>
+<label x="172.72" y="231.14" size="1.27" layer="95" rot="R180" xref="yes"/>
 </segment>
 </net>
@@
 </segment>
 <segment>
-<pinref part="J4" gate="G$1" pin="5"/>
-<wire x1="106.68" y1="185.42" x2="109.22" y2="185.42" width="0.1524" layer="91"/>
-<label x="109.22" y="185.42" size="1.27" layer="95" xref="yes"/>
+<pinref part="J4" gate="G$1" pin="4"/>
+<wire x1="106.68" y1="182.88" x2="109.22" y2="182.88" width="0.1524" layer="91"/>
+<label x="109.22" y="182.88" size="1.27" layer="95" xref="yes"/>
 </segment>
 </net>
@@
 </segment>
 <segment>
-<pinref part="IC2" gate="G$1" pin="B4"/>
-<wire x1="200.66" y1="228.6" x2="205.74" y2="228.6" width="0.1524" layer="91"/>
-<label x="205.74" y="228.6" size="1.27" layer="95" xref="yes"/>
+<pinref part="IC2" gate="G$1" pin="B3"/>
+<wire x1="200.66" y1="231.14" x2="203.2" y2="231.14" width="0.1524" layer="91"/>
+<label x="203.2" y="231.14" size="1.27" layer="95" xref="yes"/>
 </segment>
 </net>
@@
 </segment>
 </net>
+<net name="LTE_DTR" class="0">
+<segment>
+<pinref part="U1" gate="G$1" pin="DTR"/>
+<wire x1="284.48" y1="200.66" x2="281.94" y2="200.66" width="0.1524" layer="91"/>
+<label x="281.94" y="200.66" size="1.27" layer="95" rot="R180" xref="yes"/>
+</segment>
+<segment>
+<pinref part="IC2" gate="G$1" pin="A4"/>
+<wire x1="175.26" y1="228.6" x2="172.72" y2="228.6" width="0.1524" layer="91"/>
+<label x="172.72" y="228.6" size="1.27" layer="95" rot="R180" xref="yes"/>
+</segment>
+</net>
+<net name="UC_DTR" class="0">
+<segment>
+<pinref part="IC2" gate="G$1" pin="B4"/>
+<wire x1="200.66" y1="228.6" x2="203.2" y2="228.6" width="0.1524" layer="91"/>
+<label x="203.2" y="228.6" size="1.27" layer="95" xref="yes"/>
+</segment>
+<segment>
+<pinref part="J4" gate="G$1" pin="5"/>
+<wire x1="106.68" y1="185.42" x2="109.22" y2="185.42" width="0.1524" layer="91"/>
+<label x="109.22" y="185.42" size="1.27" layer="95" xref="yes"/>
+</segment>
+</net>
+<net name="N$12" class="0">
+<segment>
+<pinref part="JP3" gate="G$1" pin="2"/>
+<wire x1="254" y1="55.88" x2="256.54" y2="55.88" width="0.1524" layer="91"/>
+<pinref part="LED3" gate="G$1" pin="A"/>
+<wire x1="256.54" y1="55.88" x2="256.54" y2="53.34" width="0.1524" layer="91"/>
+</segment>
+</net>
