File: PCB Files/LTE Shield v3.brd (EAGLE design)
At the start: 58.4 x 53.3 mm, 44 parts, among them IC1 MIC5216-4.0YM5, IC2 TXB0104, IC3 MCP9808, J6 microUSB, Q1 FDV301N, Q2 FDV301N, X1 LTE-uFL, X2 GNSS-uFL

Commit message: Add files via upload
Parts:
- moved JP1 3.81 mm to (17.8, 7.75)
- moved R1 2.54 mm to (17.8, 10.9)
Connections:
- net 5V: now also R1.1; no longer JP1.1
- net EN: now also JP1.2; no longer R1.2
- net N$6: now also JP1.1, R1.2; no longer JP1.2, R1.1
Changed lines of the file:
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@@
 Released under CC-BY-SA-4.0 license</text>
 <text x="18.415" y="4.318" size="1.27" layer="21" font="vector" ratio="16" rot="R90">EN</text>
-<text x="19.05" y="12.192" size="1.016" layer="21" font="vector" ratio="16" rot="R270">EN</text>
+<text x="16.256" y="7.112" size="1.016" layer="21" font="vector" ratio="16" rot="R90">EN</text>
 <text x="4.445" y="45.085" size="1.27" layer="21" font="vector" ratio="16">SCL</text>
 <text x="4.445" y="42.545" size="1.27" layer="21" font="vector" ratio="16">SDA</text>
@@
 </element>
 <element name="C10" library="TimWoo-Capacitors" library_urn="urn:adsk.eagle:library:500759" package="1206" package3d_urn="urn:adsk.eagle:package:500778/1" value="150uF" x="38.227" y="24.892" smashed="yes" rot="MR90">
-<attribute name="NAME" x="39.116" y="27.559" size="0.8128" layer="26" font="vector" ratio="16" rot="MR0"/>
+<attribute name="NAME" x="39.116" y="27.94" size="0.8128" layer="26" font="vector" ratio="16" rot="MR0"/>
 <attribute name="VALUE" x="36.703" y="23.495" size="0.4064" layer="28" rot="MR90"/>
 </element>
 <element name="C11" library="TimWoo-Capacitors" library_urn="urn:adsk.eagle:library:500759" package="1206" package3d_urn="urn:adsk.eagle:package:500778/1" value="150uF" x="35.052" y="24.892" smashed="yes" rot="MR90">
-<attribute name="NAME" x="35.941" y="27.559" size="0.8128" layer="26" font="vector" ratio="16" rot="MR0"/>
+<attribute name="NAME" x="35.941" y="27.94" size="0.8128" layer="26" font="vector" ratio="16" rot="MR0"/>
 <attribute name="VALUE" x="33.528" y="23.495" size="0.4064" layer="28" rot="MR90"/>
 </element>
@@
 <attribute name="VALUE" x="28.067" y="10.16" size="0.4064" layer="27" font="vector" ratio="16" rot="R270"/>
 </element>
-<element name="R1" library="TimWoo-Resistors" library_urn="urn:adsk.eagle:library:500711" package="0603-RES-MARKED" package3d_urn="urn:adsk.eagle:package:500751/2" value="150k" x="17.78" y="8.382" smashed="yes" rot="R270">
-<attribute name="NAME" x="16.891" y="8.255" size="0.8128" layer="25" font="vector" ratio="16" rot="R90"/>
-<attribute name="VALUE" x="16.51" y="9.398" size="0.4064" layer="27" font="vector" ratio="16" rot="R270"/>
-</element>
-<element name="JP1" library="TimWoo-Connectors" library_urn="urn:adsk.eagle:library:1036184" package="SMT-JUMPER_2_NC_TRACE_SILK" package3d_urn="urn:adsk.eagle:package:1036528/1" value="" x="17.78" y="11.557" smashed="yes" rot="R270">
-<attribute name="NAME" x="16.51" y="11.557" size="0.6096" layer="25" font="vector" ratio="20" rot="R90" align="bottom-center"/>
-<attribute name="VALUE" x="16.637" y="11.557" size="0.6096" layer="27" font="vector" ratio="20" rot="R270" align="top-center"/>
+<element name="R1" library="TimWoo-Resistors" library_urn="urn:adsk.eagle:library:500711" package="0603-RES-MARKED" package3d_urn="urn:adsk.eagle:package:500751/2" value="150k" x="17.78" y="10.922" smashed="yes" rot="R270">
+<attribute name="NAME" x="16.891" y="10.795" size="0.8128" layer="25" font="vector" ratio="16" rot="R90"/>
+<attribute name="VALUE" x="16.51" y="11.938" size="0.4064" layer="27" font="vector" ratio="16" rot="R270"/>
+</element>
+<element name="JP1" library="TimWoo-Connectors" library_urn="urn:adsk.eagle:library:1036184" package="SMT-JUMPER_2_NC_TRACE_SILK" package3d_urn="urn:adsk.eagle:package:1036528/1" value="" x="17.78" y="7.747" smashed="yes" rot="R270">
+<attribute name="NAME" x="16.383" y="6.35" size="0.6096" layer="25" font="vector" ratio="20" rot="R180" align="bottom-center"/>
+<attribute name="VALUE" x="16.637" y="7.747" size="0.6096" layer="27" font="vector" ratio="20" rot="R270" align="top-center"/>
 </element>
 <element name="J3" library="TimWoo-Connectors" library_urn="urn:adsk.eagle:library:1036184" package="1X04_ROUND" value="" x="2.54" y="41.91" smashed="yes" rot="R270">
@@
 <contactref element="IC1" pad="1"/>
 <wire x1="27.94" y1="2.54" x2="27.94" y2="4.191" width="0.8128" layer="1"/>
-<wire x1="24.3205" y1="7.8105" x2="20.955" y2="11.176" width="0.8128" layer="1"/>
-<contactref element="JP1" pad="1"/>
+<wire x1="20.955" y1="11.176" x2="24.3205" y2="7.8105" width="0.8128" layer="1"/>
 <wire x1="24.3205" y1="7.8105" x2="27.94" y2="4.191" width="0.8128" layer="1"/>
-<wire x1="17.78" y1="12.065" x2="20.066" y2="12.065" width="0.3048" layer="1"/>
-<wire x1="20.066" y1="12.065" x2="20.955" y2="11.176" width="0.3048" layer="1"/>
 <wire x1="29.3069" y1="9.713" x2="27.659" y2="9.713" width="0.8128" layer="1"/>
 <wire x1="27.659" y1="9.713" x2="27.559" y2="9.613" width="0.8128" layer="1"/>
@@
 <wire x1="2.54" y1="38.1" x2="19.685" y2="38.1" width="0.4064" layer="16"/>
 <wire x1="19.685" y1="38.1" x2="20.955" y2="36.83" width="0.4064" layer="16"/>
+<contactref element="R1" pad="1"/>
+<wire x1="17.78" y1="11.772" x2="20.359" y2="11.772" width="0.3048" layer="1"/>
+<wire x1="20.359" y1="11.772" x2="20.955" y2="11.176" width="0.3048" layer="1"/>
 </signal>
 <signal name="SDA">
@@
 <contactref element="IC1" pad="3"/>
 <contactref element="J1" pad="8"/>
-<contactref element="R1" pad="2"/>
-<wire x1="17.78" y1="2.54" x2="17.78" y2="7.532" width="0.3048" layer="1"/>
 <wire x1="17.78" y1="2.54" x2="21.844" y2="6.604" width="0.3048" layer="16"/>
 <wire x1="21.844" y1="6.604" x2="28.956" y2="6.604" width="0.3048" layer="16"/>
@@
 <wire x1="28.956" y1="6.604" x2="29.3069" y2="6.9549" width="0.3048" layer="1"/>
 <wire x1="29.3069" y1="6.9549" x2="29.3069" y2="7.813" width="0.3048" layer="1"/>
+<contactref element="JP1" pad="2"/>
+<wire x1="17.78" y1="2.54" x2="17.78" y2="7.239" width="0.3048" layer="1"/>
 </signal>
 <signal name="N$6">
-<contactref element="JP1" pad="2"/>
-<contactref element="R1" pad="1"/>
-<wire x1="17.78" y1="9.232" x2="17.78" y2="11.049" width="0.3048" layer="1"/>
+<contactref element="R1" pad="2"/>
+<contactref element="JP1" pad="1"/>
+<wire x1="17.78" y1="8.255" x2="17.78" y2="10.072" width="0.3048" layer="1"/>
 </signal>
 </signals>

Commit message: Add files via upload
Parts:
- IC1: value MIC5216-4.0YM5 -> MIC5219-3.6YM5
Connections:
- net 4V renamed VIN
Changed lines of the file:
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@@
 <attribute name="VALUE" x="45.72" y="43.942" size="0.6096" layer="27" font="vector" ratio="20" rot="R180" align="top-center"/>
 </element>
-<element name="IC1" library="TimWoo-IC" library_urn="urn:adsk.eagle:library:500796" package="SOT23-5" package3d_urn="urn:adsk.eagle:package:500846/2" value="MIC5216-4.0YM5" x="30.607" y="8.763" smashed="yes" rot="R270">
+<element name="IC1" library="TimWoo-IC" library_urn="urn:adsk.eagle:library:500796" package="SOT23-5" package3d_urn="urn:adsk.eagle:package:500846/2" value="MIC5219-3.6YM5" x="30.607" y="8.763" smashed="yes" rot="R270">
 <attribute name="NAME" x="29.972" y="10.668" size="0.8128" layer="25" font="vector" ratio="16"/>
 <attribute name="VALUE" x="28.067" y="10.16" size="0.4064" layer="27" font="vector" ratio="16" rot="R270"/>
@@
 <contactref element="J3" pad="3"/>
 </signal>
-<signal name="4V">
+<signal name="VIN">
 <contactref element="C2" pad="1"/>
 <contactref element="U1" pad="56"/>
