File: PCB Files/LTE Shield v3.sch (EAGLE design)
At the start: 44 parts, among them IC1 MIC5216-4.0YM5, IC2 TXB0104, IC3 MCP9808, J6 microUSB, Q1 FDV301N, Q2 FDV301N, X1 LTE-uFL, X2 GNSS-uFL

Commit message: Add files via upload
Connections:
- net 5V: now also R1.1; no longer JP1.1
- net EN: now also JP1.2; no longer R1.2
- net N$6: now also JP1.1, R1.2; no longer JP1.2, R1.1
Other:
- moved on the sheet: JP1, R1
Changed lines of the file:
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@@
 than the LTE shield. If you are concerned about low
 power, please select or design a board wisely!</text>
-<text x="40.64" y="27.94" size="1.778" layer="97">Cut jumper to
+<text x="50.8" y="30.48" size="1.778" layer="97">Cut jumper to
 disable pull-up
 on EN pin</text>
@@
 <instance part="JP3" gate="G$1" x="160.02" y="63.5"/>
 <instance part="IC1" gate="G$1" x="83.82" y="43.18"/>
-<instance part="R1" gate="G$1" x="58.42" y="40.64"/>
-<instance part="JP1" gate="G$1" x="45.72" y="40.64"/>
+<instance part="R1" gate="G$1" x="45.72" y="40.64"/>
+<instance part="JP1" gate="G$1" x="58.42" y="40.64"/>
 <instance part="J3" gate="G$1" x="71.12" y="114.3"/>
 <instance part="GND4" gate="1" x="91.44" y="116.84" rot="R90"/>
@@
 <wire x1="38.1" y1="40.64" x2="38.1" y2="45.72" width="0.1524" layer="91"/>
 <junction x="38.1" y="45.72"/>
-<pinref part="JP1" gate="G$1" pin="1"/>
+<pinref part="R1" gate="G$1" pin="1"/>
 <wire x1="40.64" y1="40.64" x2="38.1" y2="40.64" width="0.1524" layer="91"/>
 </segment>
@@
 <label x="68.58" y="43.18" size="1.778" layer="95"/>
 <wire x1="66.04" y1="40.64" x2="66.04" y2="43.18" width="0.1524" layer="91"/>
-<pinref part="R1" gate="G$1" pin="2"/>
+<pinref part="JP1" gate="G$1" pin="2"/>
 <wire x1="63.5" y1="40.64" x2="66.04" y2="40.64" width="0.1524" layer="91"/>
 </segment>
@@
 <net name="N$6" class="0">
 <segment>
-<pinref part="JP1" gate="G$1" pin="2"/>
-<pinref part="R1" gate="G$1" pin="1"/>
+<pinref part="R1" gate="G$1" pin="2"/>
+<pinref part="JP1" gate="G$1" pin="1"/>
 <wire x1="50.8" y1="40.64" x2="53.34" y2="40.64" width="0.1524" layer="91"/>
 </segment>

Commit message: Add files via upload
Parts:
- IC1: value MIC5216-4.0YM5 -> MIC5219-3.6YM5
Connections:
- net 4V renamed VIN
Other:
- note added: "3.6V/500mA Regulator EN = LOW: 0.1uA + 33uA (through R1) EN = HIGH: 350uA @ 50mA draw 1.8mA @ 150mA draw"
- note added: "Set LOW to turn off the regulator"
- note removed: "4V/500mA Regulator EN = LOW: 0.1uA + 33uA (through R1) EN = HIGH: 350uA @ 50mA draw 1.8mA @ 150mA draw"
- note removed: "Set LOW to turn off 4V regulator (~0.1uA quiescent)"
Changed lines of the file:
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@@
 <part name="C2" library="TimWoo-Capacitors" deviceset="CAP" device="MARKED-0603" value="4.7uF"/>
 <part name="J6" library="TimWoo-Connectors" library_urn="urn:adsk.eagle:library:1036184" deviceset="MICRO-USB_SMD_NOSHIELD" device="V1" package3d_urn="urn:adsk.eagle:package:1036780/2" value="microUSB"/>
-<part name="SUPPLY4" library="TimWoo-Aesthetics" library_urn="urn:adsk.eagle:library:502097" deviceset="4V" device=""/>
+<part name="SUPPLY4" library="TimWoo-Aesthetics" library_urn="urn:adsk.eagle:library:502097" deviceset="VIN" device=""/>
 <part name="SUPPLY14" library="TimWoo-Aesthetics" deviceset="V_USB" device=""/>
 <part name="FID2" library="TimWoo-Aesthetics" library_urn="urn:adsk.eagle:library:502097" deviceset="FIDUCIAL" device="" package3d_urn="urn:adsk.eagle:package:502130/2"/>
@@
 <part name="GND18" library="TimWoo-Aesthetics" deviceset="GND" device=""/>
 <part name="X1" library="adafruit" library_urn="urn:adsk.eagle:library:420" deviceset="ANTENNA_U.FL" device="" value="LTE-uFL"/>
-<part name="SUPPLY17" library="TimWoo-Aesthetics" library_urn="urn:adsk.eagle:library:502097" deviceset="4V" device=""/>
+<part name="SUPPLY17" library="TimWoo-Aesthetics" library_urn="urn:adsk.eagle:library:502097" deviceset="VIN" device=""/>
 <part name="X3" library="TimWoo-Connectors" library_urn="urn:adsk.eagle:library:1036184" deviceset="MICROSIM_SOCKET_PUSH-PULL" device="" package3d_urn="urn:adsk.eagle:package:1036783/2"/>
 <part name="GND25" library="TimWoo-Aesthetics" deviceset="GND" device=""/>
@@
 <part name="C9" library="TimWoo-Capacitors" library_urn="urn:adsk.eagle:library:500759" deviceset="CAP" device="MARKED-0603" package3d_urn="urn:adsk.eagle:package:500792/2" value="1uF"/>
 <part name="C8" library="TimWoo-Capacitors" deviceset="CAP" device="MARKED-0603" package3d_urn="urn:adsk.eagle:package:500792/2" value="0.1uF"/>
-<part name="SUPPLY18" library="TimWoo-Aesthetics" library_urn="urn:adsk.eagle:library:502097" deviceset="4V" device=""/>
+<part name="SUPPLY18" library="TimWoo-Aesthetics" library_urn="urn:adsk.eagle:library:502097" deviceset="VIN" device=""/>
 <part name="SUPPLY16" library="TimWoo-Aesthetics" deviceset="V_USB" device=""/>
 <part name="C10" library="TimWoo-Capacitors" library_urn="urn:adsk.eagle:library:500759" deviceset="CAP" device="1206" package3d_urn="urn:adsk.eagle:package:500778/1" value="150uF"/>
@@
 <part name="Q1" library="TimWoo-MOSFETs" library_urn="urn:adsk.eagle:library:501962" deviceset="MOSFET-N" device="GENERIC" package3d_urn="urn:adsk.eagle:package:501973/2" value="FDV301N"/>
 <part name="Q2" library="TimWoo-MOSFETs" library_urn="urn:adsk.eagle:library:501962" deviceset="MOSFET-N" device="GENERIC" package3d_urn="urn:adsk.eagle:package:501973/2" value="FDV301N"/>
-<part name="SUPPLY5" library="TimWoo-Aesthetics" library_urn="urn:adsk.eagle:library:502097" deviceset="4V" device=""/>
-<part name="SUPPLY13" library="TimWoo-Aesthetics" library_urn="urn:adsk.eagle:library:502097" deviceset="4V" device=""/>
+<part name="SUPPLY5" library="TimWoo-Aesthetics" library_urn="urn:adsk.eagle:library:502097" deviceset="VIN" device=""/>
+<part name="SUPPLY13" library="TimWoo-Aesthetics" library_urn="urn:adsk.eagle:library:502097" deviceset="VIN" device=""/>
 <part name="JP3" library="TimWoo-Connectors" library_urn="urn:adsk.eagle:library:1036184" deviceset="JUMPER-SMT_2_NC_TRACE" device="_SILK" package3d_urn="urn:adsk.eagle:package:1036528/1"/>
-<part name="IC1" library="TimWoo-IC" library_urn="urn:adsk.eagle:library:500796" deviceset="VOLTAGE-REGULATOR_SOT23-5" device="SOT-23-5" package3d_urn="urn:adsk.eagle:package:500846/2" value="MIC5216-4.0YM5"/>
+<part name="IC1" library="TimWoo-IC" library_urn="urn:adsk.eagle:library:500796" deviceset="VOLTAGE-REGULATOR_SOT23-5" device="SOT-23-5" package3d_urn="urn:adsk.eagle:package:500846/2" value="MIC5219-3.6YM5"/>
 <part name="R1" library="TimWoo-Resistors" library_urn="urn:adsk.eagle:library:500711" deviceset="RESISTOR" device="MARKED-0603" package3d_urn="urn:adsk.eagle:package:500751/2" value="150k"/>
 <part name="JP1" library="TimWoo-Connectors" library_urn="urn:adsk.eagle:library:1036184" deviceset="JUMPER-SMT_2_NC_TRACE" device="_SILK" package3d_urn="urn:adsk.eagle:package:1036528/1"/>
@@
 <text x="144.78" y="264.16" size="5.08" layer="94">UART Logic Level Shifting</text>
 <text x="44.45" y="218.44" size="1.27" layer="91">EN</text>
-<text x="11.43" y="223.52" size="1.778" layer="97">Set LOW to turn
-off 4V regulator
-(~0.1uA quiescent)</text>
+<text x="13.97" y="223.52" size="1.778" layer="97">Set LOW to turn
+off the regulator</text>
 <wire x1="137.16" y1="99.06" x2="233.68" y2="99.06" width="0.1524" layer="94" style="longdash"/>
 <wire x1="137.16" y1="279.4" x2="137.16" y2="195.58" width="0.1524" layer="94" style="longdash"/>
@@
 disable PWR LED</text>
 <wire x1="137.16" y1="99.06" x2="137.16" y2="0" width="0.1524" layer="94" style="longdash"/>
-<text x="60.96" y="53.34" size="1.778" layer="97">4V/500mA Regulator
+<text x="60.96" y="53.34" size="1.778" layer="97">3.6V/500mA Regulator
 EN = LOW: 0.1uA + 33uA (through R1)
 EN = HIGH: 350uA @ 50mA draw
@@
 </segment>
 </net>
-<net name="4V" class="0">
+<net name="VIN" class="0">
 <segment>
 <wire x1="106.68" y1="43.18" x2="106.68" y2="45.72" width="0.1524" layer="91"/>
@@
 <pinref part="C2" gate="G$1" pin="1"/>
 <junction x="106.68" y="45.72"/>
-<pinref part="SUPPLY4" gate="G$1" pin="4V"/>
+<pinref part="SUPPLY4" gate="G$1" pin="VIN"/>
 <wire x1="106.68" y1="50.8" x2="106.68" y2="45.72" width="0.1524" layer="91"/>
 <pinref part="IC1" gate="G$1" pin="OUT"/>
@@
 <wire x1="330.2" y1="218.44" x2="330.2" y2="226.06" width="0.1524" layer="91"/>
 <wire x1="330.2" y1="226.06" x2="327.66" y2="226.06" width="0.1524" layer="91"/>
-<pinref part="SUPPLY17" gate="G$1" pin="4V"/>
+<pinref part="SUPPLY17" gate="G$1" pin="VIN"/>
 <wire x1="327.66" y1="228.6" x2="327.66" y2="226.06" width="0.1524" layer="91"/>
 </segment>
@@
 <wire x1="406.4" y1="228.6" x2="396.24" y2="228.6" width="0.1524" layer="91"/>
 <junction x="396.24" y="228.6"/>
-<pinref part="SUPPLY18" gate="G$1" pin="4V"/>
+<pinref part="SUPPLY18" gate="G$1" pin="VIN"/>
 <wire x1="391.16" y1="231.14" x2="391.16" y2="228.6" width="0.1524" layer="91"/>
 <junction x="391.16" y="228.6"/>
@@
 <segment>
 <pinref part="LED2" gate="G$1" pin="A"/>
-<pinref part="SUPPLY13" gate="G$1" pin="4V"/>
+<pinref part="SUPPLY13" gate="G$1" pin="VIN"/>
 <wire x1="208.28" y1="63.5" x2="208.28" y2="60.96" width="0.1524" layer="91"/>
 </segment>
@@
 <pinref part="JP3" gate="G$1" pin="1"/>
 <wire x1="154.94" y1="63.5" x2="152.4" y2="63.5" width="0.1524" layer="91"/>
-<pinref part="SUPPLY5" gate="G$1" pin="4V"/>
+<pinref part="SUPPLY5" gate="G$1" pin="VIN"/>
 <wire x1="152.4" y1="63.5" x2="152.4" y2="68.58" width="0.1524" layer="91"/>
 </segment>
