File: PCB Files/SIM7000 Shield v4.brd (EAGLE design)
At the start: 58.4 x 53.3 mm, 45 parts, among them IC1 MIC5219-3.6YM5, IC2 TXB0104, IC3 MCP9808, J6 microUSB, Q1 FDV301N, Q2 FDV301N, X1 LTE-uFL, X2 GNSS-uFL

Commit message: Add files via upload
Parts:
- added J7: V_logic, TimWoo-Connectors:1X02
- added JP5: (no value), TimWoo-Connectors:SMT-JUMPER_3_1-NC_TRACE_SILK
- C10, C11: device TimWoo-Capacitors:1206 -> TimWoo-Capacitors:1210
- Q1, Q2: value FDV301N -> BSS138L
- moved C10 1.37 mm to (42.0, 25.4)
- moved C11 0.63 mm to (37.2, 25.4)
Connections:
- new net N$13: J7.2, JP5.1
- new net V_LOGIC: C4.1, IC2.14, JP5.2
- net 5V: now also JP5.3; no longer C4.1, IC2.14
- net GND: now also J7.1
Routing:
- net V_LOGIC: track 0.00 -> 11.0 mm, vias 0 -> 1
- net 5V: track 101.0 -> 91.8 mm, vias 3 -> 2
- net N$13: track 0.00 -> 2.79 mm
- net VIN: track 70.3 -> 71.5 mm
Other:
- board text added: "-VCC+"
- board text added: "LOGIC"
- board text added: "SIM7000 Shield"
- board text added: "VCC"
- board text added: "v4"
- board text removed: "LTE Shield v4"

Commit message: Add files via upload
Parts:
- J6: value microUSB -> V_logic; device TimWoo-Connectors:USB-B-MICRO-SMD -> TimWoo-Connectors:1X02
- J7: value V_logic -> microUSB; device TimWoo-Connectors:1X02 -> TimWoo-Connectors:USB-B-MICRO-SMD
- JP3: device TimWoo-Connectors:SMT-JUMPER_2_NC_TRACE_SILK -> TimWoo-Connectors:SMT-JUMPER_2_NO_SILK
- JP4: device TimWoo-Connectors:SMT-JUMPER_2_NO_SILK -> TimWoo-Connectors:SMT-JUMPER_2_NC_TRACE_SILK
- moved J6 20.5 mm to (19.1, 41.9)
- moved J7 20.5 mm to (2.03, 30.5)
- moved JP3 9.96 mm to (36.6, 46.7), turned to 270 degrees
- moved JP4 9.96 mm to (45.7, 42.8), turned to 180 degrees
Connections:
- net D+: now also J7.D+; no longer J6.D+
- net D-: now also J7.D-; no longer J6.D-
- net GND: now also J6.1, J7.GND, J7.SHIELD1, J7.SHIELD2, J7.SHIELD3, J7.SHIELD4; no longer J6.GND, J6.SHIELD1, J6.SHIELD2, J6.SHIELD3, J6.SHIELD4, J7.1
- net N$12: now also JP4.2; no longer JP3.2
- net N$13: now also J6.2; no longer J7.2
- net N$8: now also JP3.1; no longer JP4.1
- net UC_DTR: now also JP3.2; no longer JP4.2
- net VIN: now also JP4.1; no longer JP3.1
- net V_USB: now also J7.VBUS; no longer J6.VBUS
Routing:
- net 5V: track 91.8 -> 93.4 mm
Changed lines of the file:
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@@
 <element name="FID2" library="TimWoo-Aesthetics" library_urn="urn:adsk.eagle:library:502097" package="FIDUCIAL_1MM" package3d_urn="urn:adsk.eagle:package:502130/2" value="FIDUCIAL" x="6.35" y="6.35" smashed="yes"/>
 <element name="FID1" library="TimWoo-Aesthetics" library_urn="urn:adsk.eagle:library:502097" package="FIDUCIAL_1MM" package3d_urn="urn:adsk.eagle:package:502130/2" value="FIDUCIAL" x="48.26" y="44.45" smashed="yes"/>
-<element name="J6" library="TimWoo-Connectors" library_urn="urn:adsk.eagle:library:1036184" package="USB-B-MICRO-SMD" package3d_urn="urn:adsk.eagle:package:1036780/3" value="microUSB" x="2.032" y="30.48" smashed="yes">
+<element name="J7" library="TimWoo-Connectors" library_urn="urn:adsk.eagle:library:1036184" package="USB-B-MICRO-SMD" package3d_urn="urn:adsk.eagle:package:1036780/3" value="microUSB" x="2.032" y="30.48" smashed="yes">
 <attribute name="NAME" x="3.556" y="34.925" size="0.8128" layer="25" font="vector" ratio="16"/>
 <attribute name="VALUE" x="0.762" y="35.941" size="0.4064" layer="27" font="vector" ratio="16"/>
@@
 <element name="Q1" library="TimWoo-MOSFETs" library_urn="urn:adsk.eagle:library:501962" package="SOT23-3" package3d_urn="urn:adsk.eagle:package:501973/2" value="BSS138L" x="47.244" y="36.322" rot="R90"/>
 <element name="Q2" library="TimWoo-MOSFETs" library_urn="urn:adsk.eagle:library:501962" package="SOT23-3" package3d_urn="urn:adsk.eagle:package:501973/2" value="BSS138L" x="47.117" y="14.351" rot="R270"/>
-<element name="JP3" library="TimWoo-Connectors" library_urn="urn:adsk.eagle:library:1036184" package="SMT-JUMPER_2_NC_TRACE_SILK" package3d_urn="urn:adsk.eagle:package:1036528/1" value="" x="45.72" y="42.799" smashed="yes" rot="R180">
+<element name="JP4" library="TimWoo-Connectors" library_urn="urn:adsk.eagle:library:1036184" package="SMT-JUMPER_2_NC_TRACE_SILK" package3d_urn="urn:adsk.eagle:package:1036528/1" value="" x="45.72" y="42.799" smashed="yes" rot="R180">
 <attribute name="NAME" x="47.244" y="42.799" size="0.6096" layer="25" font="vector" ratio="20" rot="R270" align="bottom-center"/>
 <attribute name="VALUE" x="45.72" y="43.942" size="0.6096" layer="27" font="vector" ratio="20" rot="R180" align="top-center"/>
@@
 <attribute name="VALUE" x="-0.635" y="46.99" size="1.27" layer="27" rot="R270"/>
 </element>
-<element name="JP4" library="TimWoo-Connectors" library_urn="urn:adsk.eagle:library:500889" package="SMT-JUMPER_2_NO_SILK" package3d_urn="urn:adsk.eagle:package:501659/1" value="" x="36.576" y="46.736" smashed="yes" rot="R270">
+<element name="JP3" library="TimWoo-Connectors" library_urn="urn:adsk.eagle:library:500889" package="SMT-JUMPER_2_NO_SILK" package3d_urn="urn:adsk.eagle:package:501659/1" value="" x="36.576" y="46.736" smashed="yes" rot="R270">
 <attribute name="NAME" x="35.306" y="46.736" size="0.6096" layer="25" font="vector" ratio="20" rot="R90" align="bottom-center"/>
 <attribute name="VALUE" x="35.433" y="46.736" size="0.6096" layer="27" font="vector" ratio="20" rot="R270" align="top-center"/>
@@
 <attribute name="VALUE" x="25.4" y="43.053" size="0.6096" layer="28" font="vector" ratio="20" rot="MR180" align="top-center"/>
 </element>
-<element name="J7" library="TimWoo-Connectors" library_urn="urn:adsk.eagle:library:1036184" package="1X02" package3d_urn="urn:adsk.eagle:package:1036544/1" value="V_logic" x="19.05" y="41.91" smashed="yes">
+<element name="J6" library="TimWoo-Connectors" library_urn="urn:adsk.eagle:library:1036184" package="1X02" package3d_urn="urn:adsk.eagle:package:1036544/1" value="V_logic" x="19.05" y="41.91" smashed="yes">
 <attribute name="VALUE" x="17.78" y="38.735" size="1.27" layer="27"/>
 </element>
@@
 <contactref element="C2" pad="2"/>
 <contactref element="C1" pad="2"/>
-<contactref element="J6" pad="GND"/>
-<contactref element="J6" pad="SHIELD1"/>
-<contactref element="J6" pad="SHIELD2"/>
-<contactref element="J6" pad="SHIELD3"/>
+<contactref element="J7" pad="GND"/>
+<contactref element="J7" pad="SHIELD1"/>
+<contactref element="J7" pad="SHIELD2"/>
+<contactref element="J7" pad="SHIELD3"/>
 <contactref element="U1" pad="18"/>
 <contactref element="U1" pad="17"/>
@@
 <via x="44.069" y="45.72" extent="1-16" drill="0.508" diameter="1.016"/>
 <via x="39.37" y="19.05" extent="1-16" drill="0.508" diameter="1.016"/>
-<contactref element="J6" pad="SHIELD4"/>
+<contactref element="J7" pad="SHIELD4"/>
 <via x="2.032" y="29.21" extent="1-16" drill="0.508" diameter="1.016"/>
 <contactref element="X3" pad="GND@1"/>
@@
 <contactref element="X3" pad="GND@5"/>
 <contactref element="X3" pad="GND@6"/>
-<contactref element="J7" pad="1"/>
+<contactref element="J6" pad="1"/>
 </signal>
 <signal name="VIN">
@@
 <wire x1="45.02" y1="21.4" x2="45.02" y2="20.955" width="1.905" layer="1"/>
 <contactref element="LED2" pad="A"/>
-<contactref element="JP3" pad="1"/>
+<contactref element="JP4" pad="1"/>
 <wire x1="42.799" y1="40.894" x2="44.704" y2="42.799" width="0.3048" layer="1"/>
 <wire x1="44.704" y1="42.799" x2="46.228" y2="42.799" width="0.3048" layer="1"/>
@@
 <signal name="V_USB">
 <contactref element="U1" pad="24"/>
-<contactref element="J6" pad="VBUS"/>
+<contactref element="J7" pad="VBUS"/>
 <wire x1="4.907" y1="31.78" x2="10.13" y2="31.78" width="0.3048" layer="1"/>
 <wire x1="14.51" y1="27.4" x2="21.02" y2="27.4" width="0.3048" layer="1"/>
@@
 </signal>
 <signal name="D-">
-<contactref element="J6" pad="D-"/>
+<contactref element="J7" pad="D-"/>
 <contactref element="U1" pad="28"/>
 <wire x1="21.02" y1="23.4" x2="15.97" y2="23.4" width="0.3048" layer="1"/>
@@
 </signal>
 <signal name="D+">
-<contactref element="J6" pad="D+"/>
+<contactref element="J7" pad="D+"/>
 <contactref element="U1" pad="27"/>
 <wire x1="21.02" y1="24.4" x2="16.24" y2="24.4" width="0.3048" layer="1"/>
@@
 <wire x1="20.359" y1="11.772" x2="20.955" y2="11.176" width="0.3048" layer="1"/>
 <contactref element="JP5" pad="3"/>
-<wire x1="20.955" y1="36.83" x2="25.4" y2="41.275" width="0.3048" layer="16"/>
-<wire x1="25.4" y1="41.275" x2="25.4" y2="41.91" width="0.3048" layer="16"/>
 <wire x1="25.4" y1="41.91" x2="26.416" y2="41.91" width="0.3048" layer="16"/>
+<wire x1="26.416" y1="41.91" x2="26.416" y2="40.386" width="0.3048" layer="16"/>
+<wire x1="22.86" y1="36.83" x2="20.955" y2="36.83" width="0.3048" layer="16"/>
+<wire x1="26.416" y1="40.386" x2="22.86" y2="36.83" width="0.3048" layer="16"/>
 </signal>
 <signal name="SDA">
@@
 <signal name="UC_DTR">
 <contactref element="IC2" pad="10"/>
-<contactref element="JP4" pad="2"/>
+<contactref element="JP3" pad="2"/>
 <wire x1="35.933" y1="44.397" x2="35.933" y2="45.077" width="0.3048" layer="1"/>
 <wire x1="36.576" y1="45.72" x2="36.576" y2="46.3296" width="0.3048" layer="1"/>
@@
 </signal>
 <signal name="N$12">
-<contactref element="JP3" pad="2"/>
+<contactref element="JP4" pad="2"/>
 <contactref element="LED1" pad="A"/>
 <wire x1="46.24" y1="40.386" x2="46.24" y2="42.787" width="0.3048" layer="1"/>
@@
 <signal name="N$8">
 <contactref element="J4" pad="1"/>
-<contactref element="JP4" pad="1"/>
+<contactref element="JP3" pad="1"/>
 <wire x1="31.496" y1="50.8" x2="31.496" y2="48.387" width="0.3048" layer="1"/>
 <wire x1="31.496" y1="48.387" x2="32.7406" y2="47.1424" width="0.3048" layer="1"/>
@@
 <signal name="N$13">
 <contactref element="JP5" pad="1"/>
-<contactref element="J7" pad="2"/>
+<contactref element="J6" pad="2"/>
 <wire x1="24.384" y1="41.91" x2="21.59" y2="41.91" width="0.3048" layer="16"/>
 </signal>

Commit message: Add files via upload
Connections:
- removed net N$13: J6.2, JP5.1
- new net VCC: C4.1, C5.1, IC2.14, IC3.8, J3.4, JP5.2, R2.2, R3.2, R5.2
- net 5V: no longer C5.1, IC3.8, J3.4, R2.2, R3.2, R5.2
- net V_LOGIC: now also J6.2, JP5.1; no longer C4.1, IC2.14, JP5.2
Routing:
- net VCC: track 0.00 -> 50.4 mm, vias 0 -> 2
- net 5V: track 93.4 -> 54.7 mm, vias 2 -> 1
- net V_LOGIC: track 11.0 -> 2.79 mm, vias 1 -> 0
- net N$13: track 2.79 -> 0.00 mm
Changed lines of the file:
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@@
 <text x="4.445" y="42.545" size="1.27" layer="21" font="vector" ratio="16">SDA</text>
 <text x="4.445" y="40.005" size="1.27" layer="21" font="vector" ratio="16">GND</text>
-<text x="4.445" y="37.465" size="1.27" layer="21" font="vector" ratio="16">5V</text>
+<text x="4.445" y="37.465" size="1.27" layer="21" font="vector" ratio="16">VCC</text>
 <text x="38.735" y="45.72" size="0.8128" layer="21" font="vector" ratio="16" rot="R90">DTR</text>
 <text x="44.831" y="44.196" size="0.8128" layer="21" font="vector" ratio="16">LED</text>
@@
 <signal name="5V">
 <contactref element="C1" pad="1"/>
-<contactref element="R3" pad="2"/>
-<contactref element="R5" pad="2"/>
-<contactref element="R2" pad="2"/>
-<wire x1="13.8929" y1="43.688" x2="13.931" y2="43.6499" width="0.3048" layer="1"/>
-<wire x1="13.931" y1="42.037" x2="13.931" y2="43.6499" width="0.3048" layer="1"/>
-<wire x1="13.97" y1="37.631" x2="14.771" y2="37.631" width="0.3048" layer="1"/>
-<wire x1="14.732" y1="42.037" x2="13.931" y2="42.037" width="0.3048" layer="1"/>
-<wire x1="14.732" y1="42.037" x2="15.24" y2="41.529" width="0.3048" layer="1"/>
-<via x="20.955" y="36.83" extent="1-16" drill="0.508" diameter="1.016"/>
-<wire x1="20.955" y1="36.83" x2="20.154" y2="37.631" width="0.3048" layer="1"/>
-<wire x1="15.24" y1="37.631" x2="20.154" y2="37.631" width="0.3048" layer="1"/>
-<wire x1="15.24" y1="37.631" x2="13.97" y2="37.631" width="0.3048" layer="1"/>
-<wire x1="15.24" y1="41.529" x2="15.24" y2="37.631" width="0.3048" layer="1"/>
 <contactref element="J1" pad="4"/>
-<contactref element="IC3" pad="8"/>
-<contactref element="C5" pad="1"/>
-<wire x1="10.627" y1="37.678" x2="10.674" y2="37.631" width="0.3048" layer="1"/>
-<wire x1="10.674" y1="37.631" x2="12.192" y2="37.631" width="0.3048" layer="1"/>
-<wire x1="12.192" y1="37.631" x2="13.97" y2="37.631" width="0.3048" layer="1"/>
 <via x="20.955" y="11.176" extent="1-16" drill="0.508" diameter="1.016"/>
-<wire x1="20.955" y1="36.83" x2="20.955" y2="11.176" width="0.508" layer="16"/>
 <contactref element="IC1" pad="1"/>
 <wire x1="27.94" y1="2.54" x2="27.94" y2="4.191" width="0.8128" layer="1"/>
@@
 <wire x1="27.559" y1="9.613" x2="26.123" y2="9.613" width="0.8128" layer="1"/>
 <wire x1="26.123" y1="9.613" x2="24.3205" y2="7.8105" width="0.8128" layer="1"/>
-<contactref element="J3" pad="4"/>
-<wire x1="2.54" y1="38.1" x2="19.685" y2="38.1" width="0.4064" layer="16"/>
-<wire x1="19.685" y1="38.1" x2="20.955" y2="36.83" width="0.4064" layer="16"/>
 <contactref element="R1" pad="1"/>
 <wire x1="17.78" y1="11.772" x2="20.359" y2="11.772" width="0.3048" layer="1"/>
 <wire x1="20.359" y1="11.772" x2="20.955" y2="11.176" width="0.3048" layer="1"/>
 <contactref element="JP5" pad="3"/>
-<wire x1="25.4" y1="41.91" x2="26.416" y2="41.91" width="0.3048" layer="16"/>
-<wire x1="26.416" y1="41.91" x2="26.416" y2="40.386" width="0.3048" layer="16"/>
-<wire x1="22.86" y1="36.83" x2="20.955" y2="36.83" width="0.3048" layer="16"/>
-<wire x1="26.416" y1="40.386" x2="22.86" y2="36.83" width="0.3048" layer="16"/>
+<wire x1="20.955" y1="11.176" x2="20.955" y2="30.988" width="0.6096" layer="16"/>
+<wire x1="26.416" y1="36.449" x2="26.416" y2="41.91" width="0.6096" layer="16"/>
+<wire x1="20.955" y1="30.988" x2="26.416" y2="36.449" width="0.6096" layer="16"/>
+<wire x1="26.416" y1="41.91" x2="25.4" y2="41.91" width="0.6096" layer="16"/>
 </signal>
 <signal name="SDA">
@@
 <wire x1="32.7406" y1="47.1424" x2="36.576" y2="47.1424" width="0.3048" layer="1"/>
 </signal>
-<signal name="V_LOGIC">
+<signal name="VCC">
+<contactref element="R2" pad="2"/>
+<contactref element="R3" pad="2"/>
+<contactref element="R5" pad="2"/>
+<contactref element="IC3" pad="8"/>
+<contactref element="C5" pad="1"/>
+<wire x1="10.627" y1="37.678" x2="10.674" y2="37.631" width="0.3048" layer="1"/>
+<wire x1="10.674" y1="37.631" x2="12.192" y2="37.631" width="0.3048" layer="1"/>
+<wire x1="12.192" y1="37.631" x2="13.97" y2="37.631" width="0.3048" layer="1"/>
+<contactref element="J3" pad="4"/>
+<wire x1="13.97" y1="37.631" x2="14.771" y2="37.631" width="0.3048" layer="1"/>
+<wire x1="14.771" y1="37.631" x2="15.24" y2="38.1" width="0.3048" layer="1"/>
+<wire x1="15.24" y1="41.656" x2="14.859" y2="42.037" width="0.3048" layer="1"/>
+<wire x1="14.859" y1="42.037" x2="13.931" y2="42.037" width="0.3048" layer="1"/>
+<wire x1="15.24" y1="38.1" x2="15.24" y2="41.656" width="0.3048" layer="1"/>
 <contactref element="C4" pad="1"/>
 <contactref element="IC2" pad="14"/>
+<contactref element="JP5" pad="2"/>
 <wire x1="33.708" y1="43.422" x2="33.159" y2="43.422" width="0.3048" layer="1"/>
 <wire x1="32.893" y1="43.688" x2="31.965" y2="43.688" width="0.3048" layer="1"/>
 <wire x1="33.159" y1="43.422" x2="32.893" y2="43.688" width="0.3048" layer="1"/>
-<contactref element="JP5" pad="2"/>
-<wire x1="25.4" y1="41.91" x2="25.4" y2="43.18" width="0.3048" layer="16"/>
-<wire x1="25.4" y1="43.18" x2="26.797" y2="44.577" width="0.3048" layer="16"/>
-<wire x1="26.797" y1="44.577" x2="28.067" y2="44.577" width="0.3048" layer="16"/>
+<wire x1="25.4" y1="41.91" x2="25.4" y2="43.561" width="0.3048" layer="16"/>
+<wire x1="25.4" y1="43.561" x2="26.416" y2="44.577" width="0.3048" layer="16"/>
+<wire x1="26.416" y1="44.577" x2="28.067" y2="44.577" width="0.3048" layer="16"/>
 <via x="28.067" y="44.577" extent="1-16" drill="0.508" diameter="1.016"/>
 <wire x1="28.067" y1="44.577" x2="31.623" y2="44.577" width="0.3048" layer="1"/>
 <wire x1="31.965" y1="44.235" x2="31.965" y2="43.688" width="0.3048" layer="1"/>
 <wire x1="31.623" y1="44.577" x2="31.965" y2="44.235" width="0.3048" layer="1"/>
-</signal>
-<signal name="N$13">
+<wire x1="2.54" y1="38.1" x2="17.78" y2="38.1" width="0.6096" layer="16"/>
+<wire x1="17.78" y1="38.1" x2="22.86" y2="38.1" width="0.6096" layer="16"/>
+<wire x1="22.86" y1="38.1" x2="25.4" y2="40.64" width="0.6096" layer="16"/>
+<wire x1="25.4" y1="40.64" x2="25.4" y2="41.91" width="0.6096" layer="16"/>
+<wire x1="15.24" y1="38.1" x2="17.78" y2="38.1" width="0.3048" layer="1"/>
+<via x="17.78" y="38.1" extent="1-16" drill="0.508" diameter="1.016"/>
+<wire x1="13.931" y1="42.037" x2="13.931" y2="43.6499" width="0.3048" layer="1"/>
+<wire x1="13.931" y1="43.6499" x2="13.8929" y2="43.688" width="0.3048" layer="1"/>
+</signal>
+<signal name="V_LOGIC">
 <contactref element="JP5" pad="1"/>
 <contactref element="J6" pad="2"/>
-<wire x1="24.384" y1="41.91" x2="21.59" y2="41.91" width="0.3048" layer="16"/>
+<wire x1="24.384" y1="41.91" x2="21.59" y2="41.91" width="0.6096" layer="16"/>
 </signal>
 </signals>
