File: PCB Files/SIM7000 Shield v4.sch (EAGLE design)
At the start: 45 parts, among them IC1 MIC5219-3.6YM5, IC2 TXB0104, IC3 MCP9808, J6 microUSB, Q1 FDV301N, Q2 FDV301N, X1 LTE-uFL, X2 GNSS-uFL

Commit message: Add files via upload
Parts:
- added J7: V_logic, TimWoo-Connectors:M02PTH
- added JP5: (no value), TimWoo-Connectors:JUMPER-SMT_3_1-NC_TRACE_SILK
- C10, C11: device TimWoo-Capacitors:CAP1206 -> TimWoo-Capacitors:CAPMARKED-1210
- Q1, Q2: value FDV301N -> BSS138L
Connections:
- new net N$13: J7.2, JP5.1
- new net V_LOGIC: C4.1, IC2.VCCB, JP5.2
- net 5V: now also JP5.3; no longer C4.1, IC2.VCCB
- net GND: now also J7.1
Other:
- note added: "5V logic by default. Cut trace and bridge jumper for other logic voltages"
- note added: "MCU logic voltage (1.8V - 5V)"
- note added: "Operating current: 200uA Shutdown current: 0.1uA"
- moved on the sheet: C3, C4, IC2

Commit message: Add files via upload
Parts:
- J6: value microUSB -> V_logic; device TimWoo-Connectors:MICRO-USB_SMD_NOSHIELDV1 -> TimWoo-Connectors:M02PTH
- J7: value V_logic -> microUSB; device TimWoo-Connectors:M02PTH -> TimWoo-Connectors:MICRO-USB_SMD_NOSHIELDV1
- JP3: device TimWoo-Connectors:JUMPER-SMT_2_NC_TRACE_SILK -> TimWoo-Connectors:JUMPER-SMT_2_NO_SILK
- JP4: device TimWoo-Connectors:JUMPER-SMT_2_NO_SILK -> TimWoo-Connectors:JUMPER-SMT_2_NC_TRACE_SILK
Connections:
- net D+: now also J7.D+; no longer J6.D+
- net D-: now also J7.D-; no longer J6.D-
- net GND: now also J6.1, J7.GND; no longer J6.GND, J7.1
- net N$12: now also JP4.2; no longer JP3.2
- net N$13: now also J6.2; no longer J7.2
- net N$8: now also JP3.1; no longer JP4.1
- net UC_DTR: now also JP3.2; no longer JP4.2
- net VIN: now also JP4.1; no longer JP3.1
- net V_USB: now also J7.VBUS; no longer J6.VBUS

Commit message: Add files via upload
Other:
- note added: "MCU logic voltage (1.8V - 5.5V)"
- note removed: "MCU logic voltage (1.8V - 5V)"
Changed lines of the file:
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@@
 Shutdown current: 0.1uA</text>
 <text x="147.32" y="246.38" size="1.778" layer="97">MCU logic voltage
-(1.8V - 5V)</text>
+(1.8V - 5.5V)</text>
 <text x="205.74" y="243.84" size="1.778" layer="97">5V logic by default.
 Cut trace and bridge

Commit message: Add files via upload
Connections:
- removed net N$13: J6.2, JP5.1
- new net VCC: C4.1, C5.1, IC2.VCCB, IC3.VDD, J3.4, JP5.2, R2.2, R3.2, R5.2
- net 5V: no longer C5.1, IC3.VDD, J3.4, R2.2, R3.2, R5.2
- net V_LOGIC: now also J6.2, JP5.1; no longer C4.1, IC2.VCCB, JP5.2
Changed lines of the file:
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@@
 <part name="R5" library="TimWoo-Resistors" library_urn="urn:adsk.eagle:library:500711" deviceset="RESISTOR" device="MARKED-0603" package3d_urn="urn:adsk.eagle:package:500751/2" value="10k"/>
 <part name="R3" library="TimWoo-Resistors" library_urn="urn:adsk.eagle:library:500711" deviceset="RESISTOR" device="MARKED-0603" package3d_urn="urn:adsk.eagle:package:500751/2" value="10k"/>
-<part name="SUPPLY9" library="TimWoo-Aesthetics" library_urn="urn:adsk.eagle:library:502097" deviceset="5V" device=""/>
-<part name="SUPPLY8" library="TimWoo-Aesthetics" library_urn="urn:adsk.eagle:library:502097" deviceset="5V" device=""/>
-<part name="SUPPLY12" library="TimWoo-Aesthetics" library_urn="urn:adsk.eagle:library:502097" deviceset="5V" device=""/>
+<part name="SUPPLY9" library="TimWoo-Aesthetics" library_urn="urn:adsk.eagle:library:502097" deviceset="VCC" device=""/>
+<part name="SUPPLY8" library="TimWoo-Aesthetics" library_urn="urn:adsk.eagle:library:502097" deviceset="VCC" device=""/>
+<part name="SUPPLY12" library="TimWoo-Aesthetics" library_urn="urn:adsk.eagle:library:502097" deviceset="VCC" device=""/>
 <part name="GND10" library="TimWoo-Aesthetics" deviceset="GND" device=""/>
 <part name="GND14" library="TimWoo-Aesthetics" deviceset="GND" device=""/>
 <part name="R2" library="TimWoo-Resistors" library_urn="urn:adsk.eagle:library:500711" deviceset="RESISTOR" device="MARKED-0603" package3d_urn="urn:adsk.eagle:package:500751/2" value="10k"/>
-<part name="SUPPLY6" library="TimWoo-Aesthetics" library_urn="urn:adsk.eagle:library:502097" deviceset="5V" device=""/>
+<part name="SUPPLY6" library="TimWoo-Aesthetics" library_urn="urn:adsk.eagle:library:502097" deviceset="VCC" device=""/>
 <part name="C5" library="TimWoo-Capacitors" deviceset="CAP" device="MARKED-0603" package3d_urn="urn:adsk.eagle:package:500792/2" value="0.1uF"/>
 <part name="GND15" library="TimWoo-Aesthetics" deviceset="GND" device=""/>
@@
 <part name="J3" library="TimWoo-Connectors" library_urn="urn:adsk.eagle:library:1036184" deviceset="M04" device="PTH-ROUND" package3d_urn="urn:adsk.eagle:package:1352189/1"/>
 <part name="GND4" library="TimWoo-Aesthetics" deviceset="GND" device=""/>
-<part name="SUPPLY3" library="TimWoo-Aesthetics" library_urn="urn:adsk.eagle:library:502097" deviceset="5V" device=""/>
+<part name="SUPPLY3" library="TimWoo-Aesthetics" library_urn="urn:adsk.eagle:library:502097" deviceset="VCC" device=""/>
 <part name="JP3" library="TimWoo-Connectors" library_urn="urn:adsk.eagle:library:500889" deviceset="JUMPER-SMT_2_NO" device="_SILK" package3d_urn="urn:adsk.eagle:package:501659/1"/>
 <part name="JP5" library="TimWoo-Connectors" library_urn="urn:adsk.eagle:library:1036184" deviceset="JUMPER-SMT_3_1-NC_TRACE" device="_SILK" package3d_urn="urn:adsk.eagle:package:1036527/1"/>
@@
 <part name="J6" library="TimWoo-Connectors" library_urn="urn:adsk.eagle:library:1036184" deviceset="M02" device="PTH" package3d_urn="urn:adsk.eagle:package:1036544/1" value="V_logic"/>
 <part name="GND11" library="TimWoo-Aesthetics" deviceset="GND" device=""/>
+<part name="SUPPLY19" library="TimWoo-Aesthetics" library_urn="urn:adsk.eagle:library:502097" deviceset="VCC" device=""/>
 </parts>
 <sheets>
@@
 <text x="147.32" y="246.38" size="1.778" layer="97">MCU logic voltage
 (1.8V - 5.5V)</text>
-<text x="205.74" y="243.84" size="1.778" layer="97">5V logic by default.
+<text x="205.74" y="248.92" size="1.778" layer="97">5V logic by default.
 Cut trace and bridge
 jumper for other
@@
 <instance part="J6" gate="G$1" x="175.26" y="243.84"/>
 <instance part="GND11" gate="1" x="185.42" y="238.76"/>
+<instance part="SUPPLY19" gate="G$1" x="205.74" y="241.3"/>
 </instances>
 <busses>
@@
 </segment>
 <segment>
-<pinref part="R3" gate="G$1" pin="2"/>
-<pinref part="SUPPLY8" gate="G$1" pin="5V"/>
-<wire x1="165.1" y1="157.48" x2="165.1" y2="160.02" width="0.1524" layer="91"/>
-</segment>
-<segment>
-<pinref part="SUPPLY9" gate="G$1" pin="5V"/>
-<pinref part="R5" gate="G$1" pin="2"/>
-<wire x1="172.72" y1="160.02" x2="172.72" y2="157.48" width="0.1524" layer="91"/>
-</segment>
-<segment>
-<pinref part="SUPPLY6" gate="G$1" pin="5V"/>
-<pinref part="R2" gate="G$1" pin="2"/>
-<wire x1="157.48" y1="160.02" x2="157.48" y2="157.48" width="0.1524" layer="91"/>
-</segment>
-<segment>
 <pinref part="J1" gate="G$1" pin="4"/>
 <pinref part="SUPPLY1" gate="G$1" pin="5V"/>
 <wire x1="25.4" y1="208.28" x2="20.32" y2="208.28" width="0.1524" layer="91"/>
 <wire x1="20.32" y1="208.28" x2="20.32" y2="210.82" width="0.1524" layer="91"/>
-</segment>
-<segment>
-<pinref part="IC3" gate="G$1" pin="VDD"/>
-<pinref part="SUPPLY12" gate="G$1" pin="5V"/>
-<wire x1="200.66" y1="144.78" x2="203.2" y2="144.78" width="0.1524" layer="91"/>
-<wire x1="203.2" y1="144.78" x2="203.2" y2="152.4" width="0.1524" layer="91"/>
-<pinref part="C5" gate="G$1" pin="1"/>
-<wire x1="203.2" y1="152.4" x2="203.2" y2="157.48" width="0.1524" layer="91"/>
-<wire x1="205.74" y1="152.4" x2="203.2" y2="152.4" width="0.1524" layer="91"/>
-<junction x="203.2" y="152.4"/>
-</segment>
-<segment>
-<pinref part="J3" gate="G$1" pin="4"/>
-<wire x1="76.2" y1="119.38" x2="78.74" y2="119.38" width="0.1524" layer="91"/>
-<pinref part="SUPPLY3" gate="G$1" pin="5V"/>
-<wire x1="78.74" y1="119.38" x2="78.74" y2="124.46" width="0.1524" layer="91"/>
 </segment>
 <segment>
@@
 </segment>
 </net>
-<net name="V_LOGIC" class="0">
-<segment>
+<net name="VCC" class="0">
+<segment>
+<pinref part="SUPPLY6" gate="G$1" pin="VCC"/>
+<pinref part="R2" gate="G$1" pin="2"/>
+<wire x1="157.48" y1="160.02" x2="157.48" y2="157.48" width="0.1524" layer="91"/>
+</segment>
+<segment>
+<pinref part="R3" gate="G$1" pin="2"/>
+<pinref part="SUPPLY8" gate="G$1" pin="VCC"/>
+<wire x1="165.1" y1="157.48" x2="165.1" y2="160.02" width="0.1524" layer="91"/>
+</segment>
+<segment>
+<pinref part="SUPPLY9" gate="G$1" pin="VCC"/>
+<pinref part="R5" gate="G$1" pin="2"/>
+<wire x1="172.72" y1="160.02" x2="172.72" y2="157.48" width="0.1524" layer="91"/>
+</segment>
+<segment>
+<pinref part="IC3" gate="G$1" pin="VDD"/>
+<pinref part="SUPPLY12" gate="G$1" pin="VCC"/>
+<wire x1="200.66" y1="144.78" x2="203.2" y2="144.78" width="0.1524" layer="91"/>
+<wire x1="203.2" y1="144.78" x2="203.2" y2="152.4" width="0.1524" layer="91"/>
+<pinref part="C5" gate="G$1" pin="1"/>
+<wire x1="203.2" y1="152.4" x2="203.2" y2="157.48" width="0.1524" layer="91"/>
+<wire x1="205.74" y1="152.4" x2="203.2" y2="152.4" width="0.1524" layer="91"/>
+<junction x="203.2" y="152.4"/>
+</segment>
+<segment>
+<pinref part="J3" gate="G$1" pin="4"/>
+<wire x1="76.2" y1="119.38" x2="78.74" y2="119.38" width="0.1524" layer="91"/>
+<pinref part="SUPPLY3" gate="G$1" pin="VCC"/>
+<wire x1="78.74" y1="119.38" x2="78.74" y2="124.46" width="0.1524" layer="91"/>
+</segment>
+<segment>
+<pinref part="SUPPLY19" gate="G$1" pin="VCC"/>
+<wire x1="205.74" y1="241.3" x2="205.74" y2="238.76" width="0.1524" layer="91"/>
 <wire x1="190.5" y1="223.52" x2="193.04" y2="223.52" width="0.1524" layer="91"/>
 <wire x1="193.04" y1="223.52" x2="193.04" y2="228.6" width="0.1524" layer="91"/>
@@
 <pinref part="IC2" gate="G$1" pin="VCCB"/>
 <pinref part="JP5" gate="G$1" pin="2"/>
-<wire x1="193.04" y1="241.3" x2="193.04" y2="228.6" width="0.1524" layer="91"/>
+<wire x1="193.04" y1="241.3" x2="193.04" y2="238.76" width="0.1524" layer="91"/>
 <junction x="193.04" y="228.6"/>
-</segment>
-</net>
-<net name="N$13" class="0">
+<wire x1="193.04" y1="238.76" x2="193.04" y2="228.6" width="0.1524" layer="91"/>
+<wire x1="205.74" y1="238.76" x2="193.04" y2="238.76" width="0.1524" layer="91"/>
+<junction x="193.04" y="238.76"/>
+</segment>
+</net>
+<net name="V_LOGIC" class="0">
 <segment>
 <pinref part="JP5" gate="G$1" pin="1"/>
