File: PCB Files/SIM7000 Shield v5.brd (EAGLE design)
At the start: 58.4 x 53.3 mm, 50 parts, among them IC1 MCP73831, IC2 TXB0104, IC3 MCP9808, J6 LiPo, J7 V_logic, J8 microUSB, Q1 BSS138L, Q2 BSS138L, X1 LTE-uFL, X2 GNSS-uFL

Commit message: Add files via upload
Parts:
- D1, D2: value 1N4148 -> 250mA/100V
- moved FID1 2.01 mm to (47.6, 46.4)
Changed lines of the file:
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@@
 <text x="17.653" y="38.989" size="1.27" layer="21" font="vector" ratio="16">-VCC+</text>
 <text x="18.034" y="43.688" size="1.27" layer="21" font="vector" ratio="16">LOGIC</text>
-<text x="8.636" y="9.906" size="1.27" layer="21" font="vector" ratio="16">+</text>
-<text x="37.973" y="8.255" size="1.016" layer="21" font="vector" ratio="16" rot="R90">DONE</text>
+<text x="8.636" y="9.398" size="1.27" layer="21" font="vector" ratio="16">+</text>
+<text x="38.1" y="8.255" size="1.016" layer="21" font="vector" ratio="16" rot="R90">DONE</text>
 <text x="18.415" y="4.318" size="1.27" layer="21" font="vector" ratio="16" rot="R90">VBAT</text>
 </plain>
@@
 <elements>
 <element name="FID2" library="TimWoo-Aesthetics" library_urn="urn:adsk.eagle:library:502097" package="FIDUCIAL_1MM" package3d_urn="urn:adsk.eagle:package:502130/2" value="FIDUCIAL" x="3.81" y="6.35" smashed="yes"/>
-<element name="FID1" library="TimWoo-Aesthetics" library_urn="urn:adsk.eagle:library:502097" package="FIDUCIAL_1MM" package3d_urn="urn:adsk.eagle:package:502130/2" value="FIDUCIAL" x="48.26" y="44.45" smashed="yes"/>
+<element name="FID1" library="TimWoo-Aesthetics" library_urn="urn:adsk.eagle:library:502097" package="FIDUCIAL_1MM" package3d_urn="urn:adsk.eagle:package:502130/2" value="FIDUCIAL" x="47.625" y="46.355" smashed="yes"/>
 <element name="J8" library="TimWoo-Connectors" library_urn="urn:adsk.eagle:library:1036184" package="USB-B-MICRO-SMD" package3d_urn="urn:adsk.eagle:package:1036780/3" value="microUSB" x="2.032" y="30.48" smashed="yes">
 <attribute name="NAME" x="3.556" y="34.925" size="0.8128" layer="25" font="vector" ratio="16"/>
@@
 <attribute name="VALUE" x="16.764" y="13.843" size="0.4064" layer="27" font="vector"/>
 </element>
-<element name="D3" library="TimWoo-Diodes" library_urn="urn:adsk.eagle:library:501758" package="SOT-353" value="MSQA6V1W5T2G" x="17.145" y="19.177" smashed="yes" rot="R180">
+<element name="D3" library="TimWoo-Diodes" library_urn="urn:adsk.eagle:library:501758" package="SOT-353" package3d_urn="urn:adsk.eagle:package:1036040/1" value="MSQA6V1W5T2G" x="17.145" y="19.177" smashed="yes" rot="R180">
 <attribute name="NAME" x="17.907" y="17.526" size="0.8128" layer="25" font="vector" ratio="16" rot="R180"/>
 <attribute name="VALUE" x="18.161" y="20.955" size="0.4064" layer="27" font="vector" ratio="16" rot="R180"/>
@@
 <attribute name="VALUE" x="32.131" y="44.831" size="0.4064" layer="27" font="vector" rot="R180"/>
 </element>
-<element name="IC2" library="TimWoo-IC" library_urn="urn:adsk.eagle:library:500796" package="VQFN-14" value="TXB0104" x="35.433" y="42.672" smashed="yes">
+<element name="IC2" library="TimWoo-IC" library_urn="urn:adsk.eagle:library:500796" package="VQFN-14" package3d_urn="urn:adsk.eagle:package:1035405/1" value="TXB0104" x="35.433" y="42.672" smashed="yes">
 <attribute name="NAME" x="37.592" y="43.942" size="0.8128" layer="25" font="vector" ratio="16"/>
 <attribute name="VALUE" x="33.528" y="39.751" size="0.4064" layer="27" font="vector" ratio="16"/>
@@
 <attribute name="VALUE" x="52.197" y="19.558" size="0.4064" layer="27" font="vector" rot="R180"/>
 </element>
-<element name="D1" library="TimWoo-Diodes" library_urn="urn:adsk.eagle:library:501758" package="SOD-323" package3d_urn="urn:adsk.eagle:package:501784/2" value="1N4148" x="41.021" y="43.18" smashed="yes" rot="R270">
+<element name="D1" library="TimWoo-Diodes" library_urn="urn:adsk.eagle:library:501758" package="SOD-323" package3d_urn="urn:adsk.eagle:package:501784/3" value="250mA/100V" x="41.021" y="43.18" smashed="yes" rot="R270">
 <attribute name="NAME" x="41.91" y="43.815" size="0.8128" layer="25" font="vector" ratio="16" rot="R270"/>
 <attribute name="PROD_ID" value="DIO-09646" x="41.021" y="43.18" size="1.778" layer="27" rot="R270" display="off"/>
 <attribute name="VALUE" x="39.624" y="44.196" size="0.4064" layer="27" rot="R270"/>
 </element>
-<element name="D2" library="TimWoo-Diodes" library_urn="urn:adsk.eagle:library:501758" package="SOD-323" package3d_urn="urn:adsk.eagle:package:501784/2" value="1N4148" x="26.035" y="43.18" smashed="yes" rot="R270">
+<element name="D2" library="TimWoo-Diodes" library_urn="urn:adsk.eagle:library:501758" package="SOD-323" package3d_urn="urn:adsk.eagle:package:501784/3" value="250mA/100V" x="26.035" y="43.18" smashed="yes" rot="R270">
 <attribute name="NAME" x="25.019" y="42.545" size="0.8128" layer="25" font="vector" ratio="16" rot="R90"/>
 <attribute name="PROD_ID" value="DIO-09646" x="26.035" y="43.18" size="1.778" layer="27" rot="R270" display="off"/>
@@
 <attribute name="VALUE" x="46.101" y="8.89" size="0.4064" layer="27"/>
 </element>
-<element name="IC3" library="TimWoo-IC" library_urn="urn:adsk.eagle:library:500796" package="8-TSSOP" package3d_urn="urn:adsk.eagle:package:1035421/1" value="MCP9808" x="9.652" y="39.878" smashed="yes" rot="R180">
+<element name="IC3" library="TimWoo-IC" library_urn="urn:adsk.eagle:library:500796" package="8-TSSOP" package3d_urn="urn:adsk.eagle:package:1035421/3" value="MCP9808" x="9.652" y="39.878" smashed="yes" rot="R180">
 <attribute name="NAME" x="7.979" y="39.743" size="0.8128" layer="25" font="vector" ratio="16" rot="R180"/>
 <attribute name="VALUE" x="11.662" y="43.958" size="0.8128" layer="27" font="vector" ratio="16" rot="R180"/>
