File: PCB Files/SIM7000 Shield v5.sch (EAGLE design)
At the start: 50 parts, among them IC1 MCP73831, IC2 TXB0104, IC3 MCP9808, J6 LiPo, J7 V_logic, J8 microUSB, Q1 BSS138L, Q2 BSS138L, X1 LTE-uFL, X2 GNSS-uFL

Commit message: Add files via upload
Parts:
- D1, D2: value 1N4148 -> 250mA/100V
Other:
- note added: "LiPo Battery Charging"
- note added: "SIM7000 Status LEDs"
- note removed: "SIM7000 Status LED's"
- note removed: "Voltage Regulation"
Changed lines of the file:
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@@
 <part name="C6" library="TimWoo-Capacitors" deviceset="CAP" device="MARKED-0603" value="0.22uF"/>
 <part name="GND25" library="TimWoo-Aesthetics" deviceset="GND" device=""/>
-<part name="D3" library="TimWoo-Diodes" library_urn="urn:adsk.eagle:library:501758" deviceset="TVS-DIODE-ARRAY-4X" device="" value="MSQA6V1W5T2G"/>
+<part name="D3" library="TimWoo-Diodes" library_urn="urn:adsk.eagle:library:501758" deviceset="TVS-DIODE-ARRAY-4X" device="" package3d_urn="urn:adsk.eagle:package:1036040/1" value="MSQA6V1W5T2G"/>
 <part name="GND26" library="TimWoo-Aesthetics" deviceset="GND" device=""/>
 <part name="SUPPLY16" library="TimWoo-Aesthetics" library_urn="urn:adsk.eagle:library:502097" deviceset="1.8V" device=""/>
@@
 <part name="SUPPLY10" library="TimWoo-Aesthetics" library_urn="urn:adsk.eagle:library:502097" deviceset="1.8V" device=""/>
 <part name="SUPPLY7" library="TimWoo-Aesthetics" library_urn="urn:adsk.eagle:library:502097" deviceset="1.8V" device=""/>
-<part name="IC2" library="TimWoo-IC" library_urn="urn:adsk.eagle:library:500796" deviceset="LEVEL_SHIFTER_TXB0104" device="TXB0104RGYR" value="TXB0104"/>
+<part name="IC2" library="TimWoo-IC" library_urn="urn:adsk.eagle:library:500796" deviceset="LEVEL_SHIFTER_TXB0104" device="TXB0104RGYR" package3d_urn="urn:adsk.eagle:package:1035405/1" value="TXB0104"/>
 <part name="C7" library="TimWoo-Capacitors" library_urn="urn:adsk.eagle:library:500759" deviceset="CAP" device="MARKED-0603" package3d_urn="urn:adsk.eagle:package:500792/2" value="33pF"/>
 <part name="GND27" library="TimWoo-Aesthetics" deviceset="GND" device=""/>
-<part name="D1" library="TimWoo-Diodes" library_urn="urn:adsk.eagle:library:501758" deviceset="DIODE" device="SOD323" package3d_urn="urn:adsk.eagle:package:501784/2" value="1N4148"/>
-<part name="D2" library="TimWoo-Diodes" library_urn="urn:adsk.eagle:library:501758" deviceset="DIODE" device="SOD323" package3d_urn="urn:adsk.eagle:package:501784/2" value="1N4148"/>
+<part name="D1" library="TimWoo-Diodes" library_urn="urn:adsk.eagle:library:501758" deviceset="DIODE" device="SOD323" package3d_urn="urn:adsk.eagle:package:501784/3" value="250mA/100V"/>
+<part name="D2" library="TimWoo-Diodes" library_urn="urn:adsk.eagle:library:501758" deviceset="DIODE" device="SOD323" package3d_urn="urn:adsk.eagle:package:501784/3" value="250mA/100V"/>
 <part name="X2" library="TimWoo-Connectors" library_urn="urn:adsk.eagle:library:1036184" deviceset="ANTENNA_U.FL" device="" package3d_urn="urn:adsk.eagle:package:1352190/1" value="GNSS-uFL"/>
 <part name="J2" library="TimWoo-Connectors" library_urn="urn:adsk.eagle:library:1036184" deviceset="M06" device="SILK_PTH" package3d_urn="urn:adsk.eagle:package:1036641/1"/>
@@
 <part name="LED3" library="TimWoo-LED" library_urn="urn:adsk.eagle:library:501982" deviceset="LED" device="0603-MARKED" package3d_urn="urn:adsk.eagle:package:502010/2" value="Blue"/>
 <part name="SUPPLY1" library="TimWoo-Aesthetics" library_urn="urn:adsk.eagle:library:502097" deviceset="5V" device=""/>
-<part name="IC3" library="TimWoo-IC" library_urn="urn:adsk.eagle:library:500796" deviceset="MCP9808" device="-MSOP" package3d_urn="urn:adsk.eagle:package:1035421/1" value="MCP9808"/>
+<part name="IC3" library="TimWoo-IC" library_urn="urn:adsk.eagle:library:500796" deviceset="MCP9808" device="-MSOP" package3d_urn="urn:adsk.eagle:package:1035421/3" value="MCP9808"/>
 <part name="R6" library="TimWoo-Resistors" library_urn="urn:adsk.eagle:library:500711" deviceset="RESISTOR" device="MARKED-0603" package3d_urn="urn:adsk.eagle:package:500751/2" value="10k"/>
 <part name="R4" library="TimWoo-Resistors" library_urn="urn:adsk.eagle:library:500711" deviceset="RESISTOR" device="MARKED-0603" package3d_urn="urn:adsk.eagle:package:500751/2" value="10k"/>
@@
 <text x="264.16" y="266.7" size="5.08" layer="94">SIM7000 / micro USB / SIM Card Interface</text>
 <text x="35.56" y="266.7" size="5.08" layer="94">Headers and Pinouts</text>
-<text x="40.64" y="86.36" size="5.08" layer="94">Voltage Regulation</text>
+<text x="35.56" y="86.36" size="5.08" layer="94">LiPo Battery Charging</text>
 <wire x1="233.68" y1="276.86" x2="233.68" y2="193.04" width="0.1524" layer="94" style="longdash"/>
 <wire x1="233.68" y1="193.04" x2="233.68" y2="99.06" width="0.1524" layer="94" style="longdash"/>
@@
 <wire x1="137.16" y1="193.04" x2="137.16" y2="99.06" width="0.1524" layer="94" style="longdash"/>
 <wire x1="137.16" y1="193.04" x2="233.68" y2="193.04" width="0.1524" layer="94" style="longdash"/>
-<text x="152.4" y="86.36" size="5.08" layer="94">SIM7000 Status LED's</text>
+<text x="152.4" y="86.36" size="5.08" layer="94">SIM7000 Status LEDs</text>
 <text x="165.1" y="66.04" size="1.778" layer="97">Cut jumper to
 disable PWR LED</text>
